File: argv_split/argv_split_kicad/argv_split_kicad.kicad_sch (KiCad schematic)
At the start: 81 parts, among them SW1 F1, SW10 F10, SW11 F11, SW12 F12, SW13 Caps, SW14 1, SW15 2, SW16 3, SW17 4, SW18 5, SW19 (, SW2 F2, SW20 ), SW21 6, SW22 7, SW23 8, SW24 9, SW25 0, SW26 Fn, SW27 Tab, SW28 Q, SW29 W, SW3 F3, SW30 E, SW31 R, SW32 T, SW33 {, SW34 }, SW35 Y, SW36 U, SW37 I, SW38 O, SW39 P, SW4 F4, SW40 =, SW5 F5, SW6 F6, SW7 F7, SW8 F8, SW9 F9

Commit message: fix(split): fix footprint
Parts:
- SW10, SW11, SW12, SW14, SW15, SW16, SW17, SW18, SW19, SW2, SW20, SW21, SW22, SW23, SW24, SW25, SW28, SW29, SW3, SW30, SW31, SW32, SW33, SW34, SW35, SW36, SW37, SW38, SW39, SW4, SW5, SW6, SW7, SW8, SW9: footprint PCM_Switch_Keyboard_Hotswap_Kailh:SW_Hotswap_Kailh_MX_Plated_1.00u -> PCM_Switch_Keyboard_Hotswap_Kailh:SW_Hotswap_Kailh_MX_1.00u
Changed lines of the file:
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@@
 			)
 		)
-		(property "Footprint" "PCM_Switch_Keyboard_Hotswap_Kailh:SW_Hotswap_Kailh_MX_Plated_1.00u"
+		(property "Footprint" "PCM_Switch_Keyboard_Hotswap_Kailh:SW_Hotswap_Kailh_MX_1.00u"
 			(at 209.55 96.52 0)
 			(hide yes)
@@
 			)
 		)
-		(property "Footprint" "PCM_Switch_Keyboard_Hotswap_Kailh:SW_Hotswap_Kailh_MX_Plated_1.00u"
+		(property "Footprint" "PCM_Switch_Keyboard_Hotswap_Kailh:SW_Hotswap_Kailh_MX_1.00u"
 			(at 184.15 96.52 0)
 			(hide yes)
@@
 			)
 		)
-		(property "Footprint" "PCM_Switch_Keyboard_Hotswap_Kailh:SW_Hotswap_Kailh_MX_Plated_1.00u"
+		(property "Footprint" "PCM_Switch_Keyboard_Hotswap_Kailh:SW_Hotswap_Kailh_MX_1.00u"
 			(at 133.35 45.72 0)
 			(hide yes)
@@
 			)
 		)
-		(property "Footprint" "PCM_Switch_Keyboard_Hotswap_Kailh:SW_Hotswap_Kailh_MX_Plated_1.00u"
+		(property "Footprint" "PCM_Switch_Keyboard_Hotswap_Kailh:SW_Hotswap_Kailh_MX_1.00u"
 			(at 374.65 45.72 0)
 			(hide yes)
@@
 			)
 		)
-		(property "Footprint" "PCM_Switch_Keyboard_Hotswap_Kailh:SW_Hotswap_Kailh_MX_Plated_1.00u"
+		(property "Footprint" "PCM_Switch_Keyboard_Hotswap_Kailh:SW_Hotswap_Kailh_MX_1.00u"
 			(at 234.95 71.12 0)
 			(hide yes)
@@
 			)
 		)
-		(property "Footprint" "PCM_Switch_Keyboard_Hotswap_Kailh:SW_Hotswap_Kailh_MX_Plated_1.00u"
+		(property "Footprint" "PCM_Switch_Keyboard_Hotswap_Kailh:SW_Hotswap_Kailh_MX_1.00u"
 			(at 234.95 96.52 0)
 			(hide yes)
@@
 			)
 		)
-		(property "Footprint" "PCM_Switch_Keyboard_Hotswap_Kailh:SW_Hotswap_Kailh_MX_Plated_1.00u"
+		(property "Footprint" "PCM_Switch_Keyboard_Hotswap_Kailh:SW_Hotswap_Kailh_MX_1.00u"
 			(at 209.55 45.72 0)
 			(hide yes)
@@
 			)
 		)
-		(property "Footprint" "PCM_Switch_Keyboard_Hotswap_Kailh:SW_Hotswap_Kailh_MX_Plated_1.00u"
+		(property "Footprint" "PCM_Switch_Keyboard_Hotswap_Kailh:SW_Hotswap_Kailh_MX_1.00u"
 			(at 323.85 71.12 0)
 			(hide yes)
@@
 			)
 		)
-		(property "Footprint" "PCM_Switch_Keyboard_Hotswap_Kailh:SW_Hotswap_Kailh_MX_Plated_1.00u"
+		(property "Footprint" "PCM_Switch_Keyboard_Hotswap_Kailh:SW_Hotswap_Kailh_MX_1.00u"
 			(at 158.75 71.12 0)
 			(hide yes)
@@
 			)
 		)
-		(property "Footprint" "PCM_Switch_Keyboard_Hotswap_Kailh:SW_Hotswap_Kailh_MX_Plated_1.00u"
+		(property "Footprint" "PCM_Switch_Keyboard_Hotswap_Kailh:SW_Hotswap_Kailh_MX_1.00u"
 			(at 158.75 45.72 0)
 			(hide yes)
@@
 			)
 		)
-		(property "Footprint" "PCM_Switch_Keyboard_Hotswap_Kailh:SW_Hotswap_Kailh_MX_Plated_1.00u"
+		(property "Footprint" "PCM_Switch_Keyboard_Hotswap_Kailh:SW_Hotswap_Kailh_MX_1.00u"
 			(at 400.05 96.52 0)
 			(hide yes)
@@
 			)
 		)
-		(property "Footprint" "PCM_Switch_Keyboard_Hotswap_Kailh:SW_Hotswap_Kailh_MX_Plated_1.00u"
+		(property "Footprint" "PCM_Switch_Keyboard_Hotswap_Kailh:SW_Hotswap_Kailh_MX_1.00u"
 			(at 260.35 71.12 0)
 			(hide yes)
@@
 			)
 		)
-		(property "Footprint" "PCM_Switch_Keyboard_Hotswap_Kailh:SW_Hotswap_Kailh_MX_Plated_1.00u"
+		(property "Footprint" "PCM_Switch_Keyboard_Hotswap_Kailh:SW_Hotswap_Kailh_MX_1.00u"
 			(at 374.65 96.52 0)
 			(hide yes)
@@
 			)
 		)
-		(property "Footprint" "PCM_Switch_Keyboard_Hotswap_Kailh:SW_Hotswap_Kailh_MX_Plated_1.00u"
+		(property "Footprint" "PCM_Switch_Keyboard_Hotswap_Kailh:SW_Hotswap_Kailh_MX_1.00u"
 			(at 425.45 96.52 0)
 			(hide yes)
@@
 			)
 		)
-		(property "Footprint" "PCM_Switch_Keyboard_Hotswap_Kailh:SW_Hotswap_Kailh_MX_Plated_1.00u"
+		(property "Footprint" "PCM_Switch_Keyboard_Hotswap_Kailh:SW_Hotswap_Kailh_MX_1.00u"
 			(at 323.85 96.52 0)
 			(hide yes)
@@
 			)
 		)
-		(property "Footprint" "PCM_Switch_Keyboard_Hotswap_Kailh:SW_Hotswap_Kailh_MX_Plated_1.00u"
+		(property "Footprint" "PCM_Switch_Keyboard_Hotswap_Kailh:SW_Hotswap_Kailh_MX_1.00u"
 			(at 450.85 96.52 0)
 			(hide yes)
@@
 			)
 		)
-		(property "Footprint" "PCM_Switch_Keyboard_Hotswap_Kailh:SW_Hotswap_Kailh_MX_Plated_1.00u"
+		(property "Footprint" "PCM_Switch_Keyboard_Hotswap_Kailh:SW_Hotswap_Kailh_MX_1.00u"
 			(at 184.15 71.12 0)
 			(hide yes)
@@
 			)
 		)
-		(property "Footprint" "PCM_Switch_Keyboard_Hotswap_Kailh:SW_Hotswap_Kailh_MX_Plated_1.00u"
+		(property "Footprint" "PCM_Switch_Keyboard_Hotswap_Kailh:SW_Hotswap_Kailh_MX_1.00u"
 			(at 234.95 45.72 0)
 			(hide yes)
@@
 			)
 		)
-		(property "Footprint" "PCM_Switch_Keyboard_Hotswap_Kailh:SW_Hotswap_Kailh_MX_Plated_1.00u"
+		(property "Footprint" "PCM_Switch_Keyboard_Hotswap_Kailh:SW_Hotswap_Kailh_MX_1.00u"
 			(at 400.05 45.72 0)
 			(hide yes)
@@
 			)
 		)
-		(property "Footprint" "PCM_Switch_Keyboard_Hotswap_Kailh:SW_Hotswap_Kailh_MX_Plated_1.00u"
+		(property "Footprint" "PCM_Switch_Keyboard_Hotswap_Kailh:SW_Hotswap_Kailh_MX_1.00u"
 			(at 133.35 96.52 0)
 			(hide yes)
@@
 			)
 		)
-		(property "Footprint" "PCM_Switch_Keyboard_Hotswap_Kailh:SW_Hotswap_Kailh_MX_Plated_1.00u"
+		(property "Footprint" "PCM_Switch_Keyboard_Hotswap_Kailh:SW_Hotswap_Kailh_MX_1.00u"
 			(at 349.25 71.12 0)
 			(hide yes)
@@
 			)
 		)
-		(property "Footprint" "PCM_Switch_Keyboard_Hotswap_Kailh:SW_Hotswap_Kailh_MX_Plated_1.00u"
+		(property "Footprint" "PCM_Switch_Keyboard_Hotswap_Kailh:SW_Hotswap_Kailh_MX_1.00u"
 			(at 374.65 71.12 0)
 			(hide yes)
@@
 			)
 		)
-		(property "Footprint" "PCM_Switch_Keyboard_Hotswap_Kailh:SW_Hotswap_Kailh_MX_Plated_1.00u"
+		(property "Footprint" "PCM_Switch_Keyboard_Hotswap_Kailh:SW_Hotswap_Kailh_MX_1.00u"
 			(at 349.25 96.52 0)
 			(hide yes)
@@
 			)
 		)
-		(property "Footprint" "PCM_Switch_Keyboard_Hotswap_Kailh:SW_Hotswap_Kailh_MX_Plated_1.00u"
+		(property "Footprint" "PCM_Switch_Keyboard_Hotswap_Kailh:SW_Hotswap_Kailh_MX_1.00u"
 			(at 476.25 45.72 0)
 			(hide yes)
@@
 			)
 		)
-		(property "Footprint" "PCM_Switch_Keyboard_Hotswap_Kailh:SW_Hotswap_Kailh_MX_Plated_1.00u"
+		(property "Footprint" "PCM_Switch_Keyboard_Hotswap_Kailh:SW_Hotswap_Kailh_MX_1.00u"
 			(at 260.35 96.52 0)
 			(hide yes)
@@
 			)
 		)
-		(property "Footprint" "PCM_Switch_Keyboard_Hotswap_Kailh:SW_Hotswap_Kailh_MX_Plated_1.00u"
+		(property "Footprint" "PCM_Switch_Keyboard_Hotswap_Kailh:SW_Hotswap_Kailh_MX_1.00u"
 			(at 133.35 71.12 0)
 			(hide yes)
@@
 			)
 		)
-		(property "Footprint" "PCM_Switch_Keyboard_Hotswap_Kailh:SW_Hotswap_Kailh_MX_Plated_1.00u"
+		(property "Footprint" "PCM_Switch_Keyboard_Hotswap_Kailh:SW_Hotswap_Kailh_MX_1.00u"
 			(at 158.75 96.52 0)
 			(hide yes)
@@
 			)
 		)
-		(property "Footprint" "PCM_Switch_Keyboard_Hotswap_Kailh:SW_Hotswap_Kailh_MX_Plated_1.00u"
+		(property "Footprint" "PCM_Switch_Keyboard_Hotswap_Kailh:SW_Hotswap_Kailh_MX_1.00u"
 			(at 450.85 71.12 0)
 			(hide yes)
@@
 			)
 		)
-		(property "Footprint" "PCM_Switch_Keyboard_Hotswap_Kailh:SW_Hotswap_Kailh_MX_Plated_1.00u"
+		(property "Footprint" "PCM_Switch_Keyboard_Hotswap_Kailh:SW_Hotswap_Kailh_MX_1.00u"
 			(at 349.25 45.72 0)
 			(hide yes)
@@
 			)
 		)
-		(property "Footprint" "PCM_Switch_Keyboard_Hotswap_Kailh:SW_Hotswap_Kailh_MX_Plated_1.00u"
+		(property "Footprint" "PCM_Switch_Keyboard_Hotswap_Kailh:SW_Hotswap_Kailh_MX_1.00u"
 			(at 450.85 45.72 0)
 			(hide yes)
@@
 			)
 		)
-		(property "Footprint" "PCM_Switch_Keyboard_Hotswap_Kailh:SW_Hotswap_Kailh_MX_Plated_1.00u"
+		(property "Footprint" "PCM_Switch_Keyboard_Hotswap_Kailh:SW_Hotswap_Kailh_MX_1.00u"
 			(at 184.15 45.72 0)
 			(hide yes)
@@
 			)
 		)
-		(property "Footprint" "PCM_Switch_Keyboard_Hotswap_Kailh:SW_Hotswap_Kailh_MX_Plated_1.00u"
+		(property "Footprint" "PCM_Switch_Keyboard_Hotswap_Kailh:SW_Hotswap_Kailh_MX_1.00u"
 			(at 400.05 71.12 0)
 			(hide yes)
@@
 			)
 		)
-		(property "Footprint" "PCM_Switch_Keyboard_Hotswap_Kailh:SW_Hotswap_Kailh_MX_Plated_1.00u"
+		(property "Footprint" "PCM_Switch_Keyboard_Hotswap_Kailh:SW_Hotswap_Kailh_MX_1.00u"
 			(at 425.45 71.12 0)
 			(hide yes)
@@
 			)
 		)
-		(property "Footprint" "PCM_Switch_Keyboard_Hotswap_Kailh:SW_Hotswap_Kailh_MX_Plated_1.00u"
+		(property "Footprint" "PCM_Switch_Keyboard_Hotswap_Kailh:SW_Hotswap_Kailh_MX_1.00u"
 			(at 209.55 71.12 0)
 			(hide yes)
@@
 			)
 		)
-		(property "Footprint" "PCM_Switch_Keyboard_Hotswap_Kailh:SW_Hotswap_Kailh_MX_Plated_1.00u"
+		(property "Footprint" "PCM_Switch_Keyboard_Hotswap_Kailh:SW_Hotswap_Kailh_MX_1.00u"
 			(at 425.45 45.72 0)
 			(hide yes)

Commit message: feat: keyboard layout
Parts:
- added D41, D42, D43, D44, D45, D46, D47, D48, D49, D50, D51, D52, D53, D54, D55, D56, D57, D58, D59, D60, D61, D62, D63, D64, D65, D66, D67, D68, D69, D70, D71, D72, D73, D74, D75, D76, D77, D78, D79, D80: D, Diode_THT:D_DO-35_SOD27_P7.62mm_Horizontal, symbol Device:D
- added SW41: Esc, PCM_Switch_Keyboard_Hotswap_Kailh:SW_Hotswap_Kailh_MX_1.50u, symbol Switch:SW_Push
- added SW42: A, PCM_Switch_Keyboard_Hotswap_Kailh:SW_Hotswap_Kailh_MX_1.00u, symbol Switch:SW_Push
- added SW43: S, PCM_Switch_Keyboard_Hotswap_Kailh:SW_Hotswap_Kailh_MX_1.00u, symbol Switch:SW_Push
- added SW44: D, PCM_Switch_Keyboard_Hotswap_Kailh:SW_Hotswap_Kailh_MX_1.00u, symbol Switch:SW_Push
- added SW45: F, PCM_Switch_Keyboard_Hotswap_Kailh:SW_Hotswap_Kailh_MX_1.00u, symbol Switch:SW_Push
- added SW46: G, PCM_Switch_Keyboard_Hotswap_Kailh:SW_Hotswap_Kailh_MX_1.00u, symbol Switch:SW_Push
- added SW47: [, PCM_Switch_Keyboard_Hotswap_Kailh:SW_Hotswap_Kailh_MX_1.00u, symbol Switch:SW_Push
- added SW48: ], PCM_Switch_Keyboard_Hotswap_Kailh:SW_Hotswap_Kailh_MX_1.00u, symbol Switch:SW_Push
- added SW49: H, PCM_Switch_Keyboard_Hotswap_Kailh:SW_Hotswap_Kailh_MX_1.00u, symbol Switch:SW_Push
- added SW50: J, PCM_Switch_Keyboard_Hotswap_Kailh:SW_Hotswap_Kailh_MX_1.00u, symbol Switch:SW_Push
- added SW51: K, PCM_Switch_Keyboard_Hotswap_Kailh:SW_Hotswap_Kailh_MX_1.00u, symbol Switch:SW_Push
- added SW52: L, PCM_Switch_Keyboard_Hotswap_Kailh:SW_Hotswap_Kailh_MX_1.00u, symbol Switch:SW_Push
- added SW53: ;, PCM_Switch_Keyboard_Hotswap_Kailh:SW_Hotswap_Kailh_MX_1.00u, symbol Switch:SW_Push
- added SW54: -, PCM_Switch_Keyboard_Hotswap_Kailh:SW_Hotswap_Kailh_MX_1.50u, symbol Switch:SW_Push
- added SW55: Shift, PCM_Switch_Keyboard_Hotswap_Kailh:SW_Hotswap_Kailh_MX_1.50u, symbol Switch:SW_Push
- added SW56: Z, PCM_Switch_Keyboard_Hotswap_Kailh:SW_Hotswap_Kailh_MX_1.00u, symbol Switch:SW_Push
- added SW57: X, PCM_Switch_Keyboard_Hotswap_Kailh:SW_Hotswap_Kailh_MX_1.00u, symbol Switch:SW_Push
- added SW58: C, PCM_Switch_Keyboard_Hotswap_Kailh:SW_Hotswap_Kailh_MX_1.00u, symbol Switch:SW_Push
- added SW59: V, PCM_Switch_Keyboard_Hotswap_Kailh:SW_Hotswap_Kailh_MX_1.00u, symbol Switch:SW_Push
- added SW60: B, PCM_Switch_Keyboard_Hotswap_Kailh:SW_Hotswap_Kailh_MX_1.00u, symbol Switch:SW_Push
- added SW61: ', PCM_Switch_Keyboard_Hotswap_Kailh:SW_Hotswap_Kailh_MX_1.00u, symbol Switch:SW_Push
- added SW62: ", PCM_Switch_Keyboard_Hotswap_Kailh:SW_Hotswap_Kailh_MX_1.00u, symbol Switch:SW_Push
- added SW63: N, PCM_Switch_Keyboard_Hotswap_Kailh:SW_Hotswap_Kailh_MX_1.00u, symbol Switch:SW_Push
- added SW64: M, PCM_Switch_Keyboard_Hotswap_Kailh:SW_Hotswap_Kailh_MX_1.00u, symbol Switch:SW_Push
- added SW65: ,, PCM_Switch_Keyboard_Hotswap_Kailh:SW_Hotswap_Kailh_MX_1.00u, symbol Switch:SW_Push
- added SW66: ., PCM_Switch_Keyboard_Hotswap_Kailh:SW_Hotswap_Kailh_MX_1.00u, symbol Switch:SW_Push
- added SW67: "/", PCM_Switch_Keyboard_Hotswap_Kailh:SW_Hotswap_Kailh_MX_1.00u, symbol Switch:SW_Push
- added SW68: RShift, PCM_Switch_Keyboard_Hotswap_Kailh:SW_Hotswap_Kailh_MX_1.50u, symbol Switch:SW_Push
- added SW69: Space, PCM_Switch_Keyboard_Hotswap_Kailh:SW_Hotswap_Kailh_MX_2.00u, symbol Switch:SW_Push
- added SW70: Backspace, PCM_Switch_Keyboard_Hotswap_Kailh:SW_Hotswap_Kailh_MX_2.00u, symbol Switch:SW_Push
- added SW71: Left, PCM_Switch_Keyboard_Hotswap_Kailh:SW_Hotswap_Kailh_MX_1.00u, symbol Switch:SW_Push
- added SW72: Down, PCM_Switch_Keyboard_Hotswap_Kailh:SW_Hotswap_Kailh_MX_1.00u, symbol Switch:SW_Push
- added SW73: Up, PCM_Switch_Keyboard_Hotswap_Kailh:SW_Hotswap_Kailh_MX_1.00u, symbol Switch:SW_Push
- added SW74: Right, PCM_Switch_Keyboard_Hotswap_Kailh:SW_Hotswap_Kailh_MX_1.00u, symbol Switch:SW_Push
- added SW75, SW80: Ctrl, PCM_Switch_Keyboard_Hotswap_Kailh:SW_Hotswap_Kailh_MX_2.00u, symbol Switch:SW_Push
- added SW76, SW79: Linux, PCM_Switch_Keyboard_Hotswap_Kailh:SW_Hotswap_Kailh_MX_2.00u, symbol Switch:SW_Push
- added SW77: alt, PCM_Switch_Keyboard_Hotswap_Kailh:SW_Hotswap_Kailh_MX_2.00u, symbol Switch:SW_Push
- added SW78: Return, PCM_Switch_Keyboard_Hotswap_Kailh:SW_Hotswap_Kailh_MX_2.00u, symbol Switch:SW_Push
Connections:
- net at SW17.1, SW31.1, SW5.1: now also SW45.1, SW59.1
- net at SW16.1, SW30.1, SW4.1: now also SW44.1, SW58.1
- net at SW14.1, SW2.1, SW28.1: now also SW42.1, SW56.1
- net at SW22.1, SW36.1, SW8.1: now also SW50.1, SW64.1, SW71.1
- net at SW18.1, SW32.1, SW6.1: now also SW46.1, SW60.1, SW75.1
- net at SW20.1, SW34.1: now also D70.1 (K), D71.1 (K), D72.1 (K), D73.1 (K), D74.1 (K), SW48.1, SW62.1, SW79.1
- net at SW12.1, SW26.1, SW40.1: now also SW54.1, SW68.1
- net at SW15.1, SW29.1, SW3.1: now also SW43.1, SW57.1
- net at SW1.1, SW13.1, SW27.1: now also SW41.1, SW55.1
- net at SW23.1, SW37.1, SW9.1: now also SW51.1, SW65.1, SW72.1
- net at SW19.1: now also SW33.1, SW47.1, SW61.1, SW76.1
- net at SW10.1, SW24.1, SW38.1: now also SW52.1, SW66.1, SW73.1
- net at SW11.1, SW25.1, SW39.1: now also SW53.1, SW67.1, SW74.1
- net at SW21.1, SW35.1, SW7.1: now also SW49.1, SW63.1, SW80.1
- new net: D58.2 (A), SW58.2
- new net: D50.2 (A), SW50.2
- new net: D49.2 (A), SW49.2
- new net: D48.1 (K), D49.1 (K), D50.1 (K), D51.1 (K), D52.1 (K), D53.1 (K), D54.1 (K)
- new net: D52.2 (A), SW52.2
- new net: D55.1 (K), D56.1 (K), D57.1 (K), D58.1 (K), D59.1 (K), D60.1 (K), D61.1 (K)
- new net: D61.2 (A), SW61.2
- new net: D66.2 (A), SW66.2
- new net: D48.2 (A), SW48.2
- new net: D62.1 (K), D63.1 (K), D64.1 (K), D65.1 (K), D66.1 (K), D67.1 (K), D68.1 (K)
- new net: D68.2 (A), SW68.2
- new net: D41.2 (A), SW41.2
- new net: D64.2 (A), SW64.2
- new net: D54.2 (A), SW54.2
- new net: D41.1 (K), D42.1 (K), D43.1 (K), D44.1 (K), D45.1 (K), D46.1 (K), D47.1 (K)
- new net: D45.2 (A), SW45.2
- new net: D53.2 (A), SW53.2
- new net: D63.2 (A), SW63.2
- new net: D74.2 (A), SW74.2
- new net: D67.2 (A), SW67.2
- new net: SW70.1, SW78.1
- new net: D70.2 (A), SW70.2
- new net: D75.2 (A), SW75.2
- new net: D62.2 (A), SW62.2
- new net: D55.2 (A), SW55.2
- new net: SW69.1, SW77.1
- new net: D69.2 (A), SW69.2
- new net: D72.2 (A), SW72.2
- new net: D78.1 (K), D79.1 (K), D80.1 (K)
- new net: D79.2 (A), SW79.2
- new net: D47.2 (A), SW47.2
- new net: D80.2 (A), SW80.2
- new net: D57.2 (A), SW57.2
- new net: D75.1 (K), D76.1 (K), D77.1 (K)
- new net: D77.2 (A), SW77.2
- new net: D51.2 (A), SW51.2
- new net: D71.2 (A), SW71.2
- new net: D43.2 (A), SW43.2
- new net: D42.2 (A), SW42.2
- new net: D65.2 (A), SW65.2
- new net: D60.2 (A), SW60.2
- new net: D44.2 (A), SW44.2
- new net: D76.2 (A), SW76.2
- new net: D73.2 (A), SW73.2
- new net: D78.2 (A), SW78.2
- new net: D59.2 (A), SW59.2
- new net: D46.2 (A), SW46.2
- new net: D56.2 (A), SW56.2
Other:
- moved on the sheet: A1, D1, D10, D11, D12, D13, D14, D15, D16, D17, D18, D19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

Commit message: feat(split): keyboard matrix
Parts:
- added A2: RIGHT_Pico, Module:RaspberryPi_Pico_Common_Unspecified, symbol MCU_Module:RaspberryPi_Pico
- A1: value RaspberryPi_Pico -> LEFT_Pico
Connections:
- net L_COL3: now reaches SW16.1, SW30.1, SW4.1, SW44.1, SW58.1
- net R_COL4: now reaches SW22.1, SW36.1, SW50.1, SW64.1, SW71.1, SW8.1
- net R_COL5: now reaches SW21.1, SW35.1, SW49.1, SW63.1, SW7.1, SW80.1
- net L_COL4: now reaches SW17.1, SW31.1, SW45.1, SW5.1, SW59.1
- net R_ROW3: now reaches D48.1 (K), D49.1 (K), D50.1 (K), D51.1 (K), D52.1 (K), D53.1 (K), D54.1 (K)
- net L_COL1: now reaches SW14.1, SW2.1, SW28.1, SW42.1, SW56.1
- net L_ROW4: now reaches D55.1 (K), D56.1 (K), D57.1 (K), D58.1 (K), D59.1 (K), D60.1 (K), D61.1 (K)
- net R_ROW0: now reaches D10.1 (K), D11.1 (K), D12.1 (K), D7.1 (K), D8.1 (K), D9.1 (K)
- net R_COL2: now reaches SW10.1, SW24.1, SW38.1, SW52.1, SW66.1, SW73.1
- net R_COL6: now reaches D70.1 (K), D71.1 (K), D72.1 (K), D73.1 (K), D74.1 (K), SW20.1, SW34.1, SW48.1, SW62.1, SW79.1
- net L_COL5: now reaches SW18.1, SW32.1, SW46.1, SW6.1, SW60.1, SW75.1
- net R_ROW4: now reaches D62.1 (K), D63.1 (K), D64.1 (K), D65.1 (K), D66.1 (K), D67.1 (K), D68.1 (K)
- net L_COL0: now reaches SW1.1, SW13.1, SW27.1, SW41.1, SW55.1
- net R_ROW1: now reaches D20.1 (K), D21.1 (K), D22.1 (K), D23.1 (K), D24.1 (K), D25.1 (K), D26.1 (K)
- net R_COL0: now reaches SW12.1, SW26.1, SW40.1, SW54.1, SW68.1
- net L_ROW3: now reaches D41.1 (K), D42.1 (K), D43.1 (K), D44.1 (K), D45.1 (K), D46.1 (K), D47.1 (K)
- net R_COL1: now reaches SW11.1, SW25.1, SW39.1, SW53.1, SW67.1, SW74.1
- net R_COL7: now reaches SW70.1, SW78.1
- net L_COL2: now reaches SW15.1, SW29.1, SW3.1, SW43.1, SW57.1
- net L_COL7: now reaches SW69.1, SW77.1
- net L_ROW1: now reaches D13.1 (K), D14.1 (K), D15.1 (K), D16.1 (K), D17.1 (K), D18.1 (K), D19.1 (K)
- net R_COL3: now reaches SW23.1, SW37.1, SW51.1, SW65.1, SW72.1, SW9.1
- net R_ROW6: now reaches D78.1 (K), D79.1 (K), D80.1 (K)
- net L_COL6: now reaches SW19.1, SW33.1, SW47.1, SW61.1, SW76.1
- net L_ROW0: now reaches D1.1 (K), D2.1 (K), D3.1 (K), D4.1 (K), D5.1 (K), D6.1 (K)
- net L_ROW6: now reaches D75.1 (K), D76.1 (K), D77.1 (K)
- net R_ROW2: now reaches D34.1 (K), D35.1 (K), D36.1 (K), D37.1 (K), D38.1 (K), D39.1 (K), D40.1 (K)
- net L_ROW2: now reaches D27.1 (K), D28.1 (K), D29.1 (K), D30.1 (K), D31.1 (K), D32.1 (K), D33.1 (K)
- net L_ROW5: now reaches D69.1 (K)
- new net: A2.13 (GND), A2.18 (GND), A2.23 (GND), A2.28 (GND), A2.3 (GND), A2.38 (GND), A2.8 (GND)
Other:
- moved on the sheet: D1, D10, D11, D12, D13, D14, D15, D16, D17, D18, D19, D2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
