File: argv_split/argv_split_kicad/argv_split_kicad.kicad_sch (KiCad schematic)
At the start: 164 parts, among them J1 Conn_01x04, J2 Conn_01x04, SW1 F1, SW10 F10, SW11 F11, SW12 F12, SW13 Caps, SW14 1, SW15 2, SW16 3, SW17 4, SW18 5, SW19 (, SW2 F2, SW20 ), SW21 6, SW22 7, SW23 8, SW24 9, SW25 0, SW26 Fn, SW27 Tab, SW28 Q, SW29 W, SW3 F3, SW30 E, SW31 R, SW32 T, SW33 {, SW34 }, SW35 Y, SW36 U, SW37 I, SW38 O, SW39 P, SW4 F4, SW40 =, SW41 Esc, SW42 A, SW43 S, SW44 D, SW45 F, SW46 G, SW47 [, SW48 ], SW49 H, SW5 F5, SW50 J, SW51 K, SW52 L, SW53 ;, SW54 -, SW55 Shift, SW56 Z, SW57 X, SW58 C, SW59 V, SW6 F6, SW60 B, SW61 ', SW62 ", SW63 N, SW64 M, SW65 ,, SW66 ., SW67 "/", SW68 RShift, SW69 Space, SW7 F7, SW70 Backspace, SW71 Left, SW72 Down, SW73 Up, SW74 Right, SW75 Ctrl, SW76 Linux, SW77 alt, SW78 Return, SW79 Linux, SW8 F8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

Commit message: refactor(argv-split): update keyboard and PCB layout
Parts:
- removed D71, D72, D73, D74: D, Diode_THT:D_DO-35_SOD27_P5.08mm_Vertical_AnodeUp, symbol Device:D
- removed SW71: Left, PCM_Switch_Keyboard_Hotswap_Kailh:SW_Hotswap_Kailh_MX_1.00u, symbol Switch:SW_Push
- removed SW72: Down, PCM_Switch_Keyboard_Hotswap_Kailh:SW_Hotswap_Kailh_MX_1.00u, symbol Switch:SW_Push
- removed SW73: Up, PCM_Switch_Keyboard_Hotswap_Kailh:SW_Hotswap_Kailh_MX_1.00u, symbol Switch:SW_Push
- removed SW74: Right, PCM_Switch_Keyboard_Hotswap_Kailh:SW_Hotswap_Kailh_MX_1.00u, symbol Switch:SW_Push
Connections:
- net R_COL7 is gone; now on net R_COL6: SW70.1, SW78.1
- net GND: now also A1.33 (AGND), A2.33 (AGND)
- net L_COL6: no longer A1.15 (GPIO11), D55.1 (K), D56.1 (K), D57.1 (K), D58.1 (K), D59.1 (K), D60.1 (K), D61.1 (K)
- net R_COL0: now also A2.1 (GPIO0)
- net R_COL1: now also A2.2 (GPIO1)
- net R_COL2: now also A2.4 (GPIO2)
- net R_COL3: now also A2.5 (GPIO3)
- net R_COL4: now also A2.6 (GPIO4), SW80.1
- net R_COL5: now also A2.7 (GPIO5), SW79.1; no longer SW80.1
- net R_COL6: now also A2.9 (GPIO6); no longer D70.1 (K), SW79.1
- net R_ROW0: now also A2.10 (GPIO7)
- net R_ROW1: now also A2.11 (GPIO8)
- net R_ROW2: now also A2.12 (GPIO9)
- net R_ROW3: now also A2.14 (GPIO10)
- net R_ROW4: now also A2.15 (GPIO11)
- net R_ROW6: now also A2.17 (GPIO13)
- net R_ROW5: now reaches A2.16 (GPIO12)
- net R_ROW5: now also D70.1 (K)
- net GPIO20 renamed L_GPIO20
- net L_GPIO20: no longer A2.26 (GPIO20), J2.2 (Pin_2)
- net GPIO21 renamed L_GPIO21
- net L_GPIO21: no longer A2.27 (GPIO21), J2.3 (Pin_3)
- new net L_ROW4: A1.15 (GPIO11), D55.1 (K), D56.1 (K), D57.1 (K), D58.1 (K), D59.1 (K), D60.1 (K), D61.1 (K)
- new net R_GPIO20: A2.26 (GPIO20), J2.2 (Pin_2)
- new net R_GPIO21: A2.27 (GPIO21), J2.3 (Pin_3)
- no-connect marks 0 -> 30
Other:
- moved on the sheet: D75, D76, D77, SW75, SW76, SW77

Commit message: feat: new layout
Parts:
- removed J1, J2: Conn_01x04, Connector_PinHeader_2.54mm:PinHeader_1x04_P2.54mm_Vertical, symbol Connector_Generic:Conn_01x04
- added J3, J4: AudioJack4, Connector_Audio:Jack_3.5mm_PJ320E_Horizontal, symbol Connector_Audio:AudioJack4
- A1, A2: now not fitted
- D1, D10, D11, D12, D13, D14, D15, D16, D17, D18, D19, D2, D20, D21, D22, D23, D24, D25, D26, D27, D28, D29, D3, D30, D31, D32, D33, D34, D35, D36, D37, D38, D39, D4, D40, D41, D42, D43, D44, D45, D46, D47, D48, D49, D5, D50, D51, D52, D53, D54, D55, D56, D57, D58, D59, D6, D60, D61, D62, D63, D64, D65, D66, D67, D68, D69, D7, D70, D8, D9: footprint Diode_THT:D_DO-35_SOD27_P5.08mm_Vertical_AnodeUp -> Diode_THT:D_DO-35_SOD27_P7.62mm_Horizontal
- D71: renamed from D75; footprint Diode_THT:D_DO-35_SOD27_P5.08mm_Vertical_AnodeUp -> Diode_THT:D_DO-35_SOD27_P7.62mm_Horizontal
- D72: renamed from D76; footprint Diode_THT:D_DO-35_SOD27_P5.08mm_Vertical_AnodeUp -> Diode_THT:D_DO-35_SOD27_P7.62mm_Horizontal
- D73: renamed from D77; footprint Diode_THT:D_DO-35_SOD27_P5.08mm_Vertical_AnodeUp -> Diode_THT:D_DO-35_SOD27_P7.62mm_Horizontal
- D74: renamed from D78; footprint Diode_THT:D_DO-35_SOD27_P5.08mm_Vertical_AnodeUp -> Diode_THT:D_DO-35_SOD27_P7.62mm_Horizontal
- D75: renamed from D79; footprint Diode_THT:D_DO-35_SOD27_P5.08mm_Vertical_AnodeUp -> Diode_THT:D_DO-35_SOD27_P7.62mm_Horizontal
- D76: renamed from D80; footprint Diode_THT:D_DO-35_SOD27_P5.08mm_Vertical_AnodeUp -> Diode_THT:D_DO-35_SOD27_P7.62mm_Horizontal
- renumbered SW75 to SW71, SW76 to SW72, SW77 to SW73, SW78 to SW74, SW79 to SW75, SW80 to SW76
Connections:
- net GND: now also J3.S, J4.S
- net L_COL0: no longer SW1.1
- net L_COL1: now also SW1.1; no longer SW2.1
- net L_COL2: now also SW2.1; no longer SW3.1
- net L_COL3: now also SW3.1; no longer SW4.1
- net L_COL4: now also SW4.1; no longer SW5.1
- net L_COL5: now also SW5.1; no longer SW6.1
- net L_COL6: now also SW6.1
- net L_GPIO20: now also J3.R1
- net L_GPIO21: now also J3.T
- net R_COL0: no longer SW12.1
- net R_COL1: now also SW12.1; no longer SW11.1
- net R_COL2: now also SW11.1; no longer SW10.1
- net R_COL3: now also SW10.1; no longer SW9.1
- net R_COL4: now also SW9.1; no longer SW8.1
- net R_COL5: now also SW8.1; no longer SW7.1
- net R_COL6: now also SW7.1
- net R_GPIO20: now also J4.R1
- net R_GPIO21: now also J4.T
- net R_VSYS: now reaches A1.39 (VSYS)
- net R_VSYS: now also J3.R2
- net VBUS: no longer names the net of A1.40 (VBUS)
- net VSYS renamed L_VSYS
- net L_VSYS: now also J4.R2
