File: argv_split/argv_split_kicad/argv_split_kicad.kicad_pcb (KiCad board)
At the start: 2 copper layers, 164 parts, among them J1 Conn_01x04, J2 Conn_01x04, SW1 F1, SW10 F10, SW11 F11, SW12 F12, SW13 Caps, SW14 1, SW15 2, SW16 3, SW17 4, SW18 5, SW19 (, SW2 F2, SW20 ), SW21 6, SW22 7, SW23 8, SW24 9, SW25 0, SW26 Fn, SW27 Tab, SW28 Q, SW29 W, SW3 F3, SW30 E, SW31 R, SW32 T, SW33 {, SW34 }, SW35 Y, SW36 U, SW37 I, SW38 O, SW39 P, SW4 F4, SW40 =, SW41 Esc, SW42 A, SW43 S, SW44 D, SW45 F, SW46 G, SW47 [, SW48 ], SW49 H, SW5 F5, SW50 J, SW51 K, SW52 L, SW53 ;, SW54 -, SW55 Shift, SW56 Z, SW57 X, SW58 C, SW59 V, SW6 F6, SW60 B, SW61 ', SW62 ", SW63 N, SW64 M, SW65 ,, SW66 ., SW67 "/", SW68 RShift, SW69 Space, SW7 F7, SW70 Backspace, SW71 Left, SW72 Down, SW73 Up, SW74 Right, SW75 Ctrl, SW76 Linux, SW77 alt, SW78 Return, SW79 Linux, SW8 F8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

Commit message: revert: starting pcb layout
Parts:
- removed A1: LEFT_Pico, Module:RaspberryPi_Pico_Common_Unspecified
- removed A2: RIGHT_Pico, Module:RaspberryPi_Pico_Common_Unspecified
- removed D1, D10, D11, D12, D13, D14, D15, D16, D17, D18, D19, D2, D20, D21, D22, D23, D24, D25, D26, D27, D28, D29, D3, D30, D31, D32, D33, D34, D35, D36, D37, D38, D39, D4, D40, D41, D42, D43, D44, D45, D46, D47, D48, D49, D5, D50, D51, D52, D53, D54, D55, D56, D57, D58, D59, D6, D60, D61, D62, D63, D64, D65, D66, D67, D68, D69, D7, D70, D71, D72, D73, D74, D75, D76, D77, D78, D79, D8, D80, D9: D, Diode_THT:D_DO-35_SOD27_P7.62mm_Horizontal
- removed J1, J2: Conn_01x04, Connector_PinHeader_2.54mm:PinHeader_1x04_P2.54mm_Vertical
- removed SW1: F1, PCM_Switch_Keyboard_Hotswap_Kailh:SW_Hotswap_Kailh_MX_1.00u
- removed SW10: F10, PCM_Switch_Keyboard_Hotswap_Kailh:SW_Hotswap_Kailh_MX_1.00u
- removed SW11: F11, PCM_Switch_Keyboard_Hotswap_Kailh:SW_Hotswap_Kailh_MX_1.00u
- removed SW12: F12, PCM_Switch_Keyboard_Hotswap_Kailh:SW_Hotswap_Kailh_MX_1.00u
- removed SW13: Caps, PCM_Switch_Keyboard_Hotswap_Kailh:SW_Hotswap_Kailh_MX_1.50u
- removed SW14: 1, PCM_Switch_Keyboard_Hotswap_Kailh:SW_Hotswap_Kailh_MX_1.00u
- removed SW15: 2, PCM_Switch_Keyboard_Hotswap_Kailh:SW_Hotswap_Kailh_MX_1.00u
- removed SW16: 3, PCM_Switch_Keyboard_Hotswap_Kailh:SW_Hotswap_Kailh_MX_1.00u
- removed SW17: 4, PCM_Switch_Keyboard_Hotswap_Kailh:SW_Hotswap_Kailh_MX_1.00u
- removed SW18: 5, PCM_Switch_Keyboard_Hotswap_Kailh:SW_Hotswap_Kailh_MX_1.00u
- removed SW19: (, PCM_Switch_Keyboard_Hotswap_Kailh:SW_Hotswap_Kailh_MX_1.00u
- removed SW2: F2, PCM_Switch_Keyboard_Hotswap_Kailh:SW_Hotswap_Kailh_MX_1.00u
- removed SW20: ), PCM_Switch_Keyboard_Hotswap_Kailh:SW_Hotswap_Kailh_MX_1.00u
- removed SW21: 6, PCM_Switch_Keyboard_Hotswap_Kailh:SW_Hotswap_Kailh_MX_1.00u
- removed SW22: 7, PCM_Switch_Keyboard_Hotswap_Kailh:SW_Hotswap_Kailh_MX_1.00u
- removed SW23: 8, PCM_Switch_Keyboard_Hotswap_Kailh:SW_Hotswap_Kailh_MX_1.00u
- removed SW24: 9, PCM_Switch_Keyboard_Hotswap_Kailh:SW_Hotswap_Kailh_MX_1.00u
- removed SW25: 0, PCM_Switch_Keyboard_Hotswap_Kailh:SW_Hotswap_Kailh_MX_1.00u
- removed SW26: Fn, PCM_Switch_Keyboard_Hotswap_Kailh:SW_Hotswap_Kailh_MX_1.50u
- removed SW27: Tab, PCM_Switch_Keyboard_Hotswap_Kailh:SW_Hotswap_Kailh_MX_1.50u
- removed SW28: Q, PCM_Switch_Keyboard_Hotswap_Kailh:SW_Hotswap_Kailh_MX_1.00u
- removed SW29: W, PCM_Switch_Keyboard_Hotswap_Kailh:SW_Hotswap_Kailh_MX_1.00u
- removed SW3: F3, PCM_Switch_Keyboard_Hotswap_Kailh:SW_Hotswap_Kailh_MX_1.00u
- removed SW30: E, PCM_Switch_Keyboard_Hotswap_Kailh:SW_Hotswap_Kailh_MX_1.00u
- removed SW31: R, PCM_Switch_Keyboard_Hotswap_Kailh:SW_Hotswap_Kailh_MX_1.00u
- removed SW32: T, PCM_Switch_Keyboard_Hotswap_Kailh:SW_Hotswap_Kailh_MX_1.00u
- removed SW33: {, PCM_Switch_Keyboard_Hotswap_Kailh:SW_Hotswap_Kailh_MX_1.00u
- removed SW34: }, PCM_Switch_Keyboard_Hotswap_Kailh:SW_Hotswap_Kailh_MX_1.00u
- removed SW35: Y, PCM_Switch_Keyboard_Hotswap_Kailh:SW_Hotswap_Kailh_MX_1.00u
- removed SW36: U, PCM_Switch_Keyboard_Hotswap_Kailh:SW_Hotswap_Kailh_MX_1.00u
- removed SW37: I, PCM_Switch_Keyboard_Hotswap_Kailh:SW_Hotswap_Kailh_MX_1.00u
- removed SW38: O, PCM_Switch_Keyboard_Hotswap_Kailh:SW_Hotswap_Kailh_MX_1.00u
- removed SW39: P, PCM_Switch_Keyboard_Hotswap_Kailh:SW_Hotswap_Kailh_MX_1.00u
- removed SW4: F4, PCM_Switch_Keyboard_Hotswap_Kailh:SW_Hotswap_Kailh_MX_1.00u
- removed SW40: =, PCM_Switch_Keyboard_Hotswap_Kailh:SW_Hotswap_Kailh_MX_1.50u
- removed SW41: Esc, PCM_Switch_Keyboard_Hotswap_Kailh:SW_Hotswap_Kailh_MX_1.50u
- removed SW42: A, PCM_Switch_Keyboard_Hotswap_Kailh:SW_Hotswap_Kailh_MX_1.00u
- removed SW43: S, PCM_Switch_Keyboard_Hotswap_Kailh:SW_Hotswap_Kailh_MX_1.00u
- removed SW44: D, PCM_Switch_Keyboard_Hotswap_Kailh:SW_Hotswap_Kailh_MX_1.00u
- removed SW45: F, PCM_Switch_Keyboard_Hotswap_Kailh:SW_Hotswap_Kailh_MX_1.00u
- removed SW46: G, PCM_Switch_Keyboard_Hotswap_Kailh:SW_Hotswap_Kailh_MX_1.00u
- removed SW47: [, PCM_Switch_Keyboard_Hotswap_Kailh:SW_Hotswap_Kailh_MX_1.00u
- removed SW48: ], PCM_Switch_Keyboard_Hotswap_Kailh:SW_Hotswap_Kailh_MX_1.00u
- removed SW49: H, PCM_Switch_Keyboard_Hotswap_Kailh:SW_Hotswap_Kailh_MX_1.00u
- removed SW5: F5, PCM_Switch_Keyboard_Hotswap_Kailh:SW_Hotswap_Kailh_MX_1.00u
- removed SW50: J, PCM_Switch_Keyboard_Hotswap_Kailh:SW_Hotswap_Kailh_MX_1.00u
- removed SW51: K, PCM_Switch_Keyboard_Hotswap_Kailh:SW_Hotswap_Kailh_MX_1.00u
- removed SW52: L, PCM_Switch_Keyboard_Hotswap_Kailh:SW_Hotswap_Kailh_MX_1.00u
- removed SW53: ;, PCM_Switch_Keyboard_Hotswap_Kailh:SW_Hotswap_Kailh_MX_1.00u
- removed SW54: -, PCM_Switch_Keyboard_Hotswap_Kailh:SW_Hotswap_Kailh_MX_1.50u
- removed SW55: Shift, PCM_Switch_Keyboard_Hotswap_Kailh:SW_Hotswap_Kailh_MX_1.50u
- removed SW56: Z, PCM_Switch_Keyboard_Hotswap_Kailh:SW_Hotswap_Kailh_MX_1.00u
- removed SW57: X, PCM_Switch_Keyboard_Hotswap_Kailh:SW_Hotswap_Kailh_MX_1.00u
- removed SW58: C, PCM_Switch_Keyboard_Hotswap_Kailh:SW_Hotswap_Kailh_MX_1.00u
- removed SW59: V, PCM_Switch_Keyboard_Hotswap_Kailh:SW_Hotswap_Kailh_MX_1.00u
- removed SW6: F6, PCM_Switch_Keyboard_Hotswap_Kailh:SW_Hotswap_Kailh_MX_1.00u
- removed SW60: B, PCM_Switch_Keyboard_Hotswap_Kailh:SW_Hotswap_Kailh_MX_1.00u
- removed SW61: ', PCM_Switch_Keyboard_Hotswap_Kailh:SW_Hotswap_Kailh_MX_1.00u
- removed SW62: ", PCM_Switch_Keyboard_Hotswap_Kailh:SW_Hotswap_Kailh_MX_1.00u
- removed SW63: N, PCM_Switch_Keyboard_Hotswap_Kailh:SW_Hotswap_Kailh_MX_1.00u
- removed SW64: M, PCM_Switch_Keyboard_Hotswap_Kailh:SW_Hotswap_Kailh_MX_1.00u
- removed SW65: ,, PCM_Switch_Keyboard_Hotswap_Kailh:SW_Hotswap_Kailh_MX_1.00u
- removed SW66: ., PCM_Switch_Keyboard_Hotswap_Kailh:SW_Hotswap_Kailh_MX_1.00u
- removed SW67: "/", PCM_Switch_Keyboard_Hotswap_Kailh:SW_Hotswap_Kailh_MX_1.00u
- removed SW68: RShift, PCM_Switch_Keyboard_Hotswap_Kailh:SW_Hotswap_Kailh_MX_1.50u
- removed SW69: Space, PCM_Switch_Keyboard_Hotswap_Kailh:SW_Hotswap_Kailh_MX_2.00u
- removed SW7: F7, PCM_Switch_Keyboard_Hotswap_Kailh:SW_Hotswap_Kailh_MX_1.00u
- removed SW70: Backspace, PCM_Switch_Keyboard_Hotswap_Kailh:SW_Hotswap_Kailh_MX_2.00u
- removed SW71: Left, PCM_Switch_Keyboard_Hotswap_Kailh:SW_Hotswap_Kailh_MX_1.00u
- removed SW72: Down, PCM_Switch_Keyboard_Hotswap_Kailh:SW_Hotswap_Kailh_MX_1.00u
- removed SW73: Up, PCM_Switch_Keyboard_Hotswap_Kailh:SW_Hotswap_Kailh_MX_1.00u
- removed SW74: Right, PCM_Switch_Keyboard_Hotswap_Kailh:SW_Hotswap_Kailh_MX_1.00u
- removed SW75, SW80: Ctrl, PCM_Switch_Keyboard_Hotswap_Kailh:SW_Hotswap_Kailh_MX_2.00u_90deg
- removed SW76, SW79: Linux, PCM_Switch_Keyboard_Hotswap_Kailh:SW_Hotswap_Kailh_MX_2.00u_90deg
- removed SW77: alt, PCM_Switch_Keyboard_Hotswap_Kailh:SW_Hotswap_Kailh_MX_2.00u_90deg
- removed SW78: Return, PCM_Switch_Keyboard_Hotswap_Kailh:SW_Hotswap_Kailh_MX_2.00u_90deg
- removed SW8: F8, PCM_Switch_Keyboard_Hotswap_Kailh:SW_Hotswap_Kailh_MX_1.00u
- removed SW9: F9, PCM_Switch_Keyboard_Hotswap_Kailh:SW_Hotswap_Kailh_MX_1.00u
Routing:
- net L_COL6: track 127.9 -> 0.00 mm
- net L_COL5: track 127.4 -> 0.00 mm
- net L_ROW2: track 123.2 -> 0.00 mm
- net L_ROW1: track 122.1 -> 0.00 mm
- net L_COL4: track 121.2 -> 0.00 mm
- net L_ROW0: track 100.0 -> 0.00 mm
- net L_COL3: track 76.2 -> 0.00 mm
- net L_COL2: track 76.2 -> 0.00 mm
- net L_COL1: track 76.2 -> 0.00 mm
- net L_COL0: track 59.1 -> 0.00 mm
- net L_ROW6: track 42.5 -> 0.00 mm
- net Net-(D75-A): track 12.0 -> 0.00 mm
- net Net-(D4-A): track 10.9 -> 0.00 mm
- net Net-(D16-A): track 10.9 -> 0.00 mm
- net Net-(D17-A): track 10.9 -> 0.00 mm
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
Commit message: feat: pcb layout
Parts:
- added A1: LEFT_Pico, Module:RaspberryPi_Pico_Common_Unspecified, F.Cu at (279.8, 166.9)
- added A2: RIGHT_Pico, Module:RaspberryPi_Pico_Common_Unspecified, B.Cu at (364.9, 166.7)
- added D1: D, Diode_THT:D_DO-35_SOD27_P5.08mm_Vertical_AnodeUp, B.Cu at (137.8, 128.6)
- added D10: D, Diode_THT:D_DO-35_SOD27_P5.08mm_Vertical_AnodeUp, B.Cu at (485.5, 125.3)
- added D11: D, Diode_THT:D_DO-35_SOD27_P5.08mm_Vertical_AnodeUp, B.Cu at (504.5, 128.9)
- added D12: D, Diode_THT:D_DO-35_SOD27_P5.08mm_Vertical_AnodeUp, B.Cu at (523.6, 128.9)
- added D13: D, Diode_THT:D_DO-35_SOD27_P5.08mm_Vertical_AnodeUp, B.Cu at (134.9, 147.6)
- added D14: D, Diode_THT:D_DO-35_SOD27_P5.08mm_Vertical_AnodeUp, B.Cu at (156.8, 147.6)
- added D15: D, Diode_THT:D_DO-35_SOD27_P5.08mm_Vertical_AnodeUp, B.Cu at (175.9, 138.8)
- added D16: D, Diode_THT:D_DO-35_SOD27_P5.08mm_Vertical_AnodeUp, B.Cu at (194.9, 138.6)
- added D17: D, Diode_THT:D_DO-35_SOD27_P5.08mm_Vertical_AnodeUp, B.Cu at (214.0, 143.4)
- added D18: D, Diode_THT:D_DO-35_SOD27_P5.08mm_Vertical_AnodeUp, B.Cu at (233.1, 147.6)
- added D19: D, Diode_THT:D_DO-35_SOD27_P5.08mm_Vertical_AnodeUp, B.Cu at (252.1, 147.6)
- added D2: D, Diode_THT:D_DO-35_SOD27_P5.08mm_Vertical_AnodeUp, B.Cu at (156.8, 128.6)
- added D20: D, Diode_THT:D_DO-35_SOD27_P5.08mm_Vertical_AnodeUp, F.Cu at (590.9, 134.7)
- added D21: D, Diode_THT:D_DO-35_SOD27_P5.08mm_Vertical_AnodeUp, F.Cu at (590.9, 138.3)
- added D22: D, Diode_THT:D_DO-35_SOD27_P5.08mm_Vertical_AnodeUp, F.Cu at (590.9, 141.8)
- added D23: D, Diode_THT:D_DO-35_SOD27_P5.08mm_Vertical_AnodeUp, F.Cu at (590.9, 145.4)
- added D24: D, Diode_THT:D_DO-35_SOD27_P5.08mm_Vertical_AnodeUp, F.Cu at (590.9, 148.9)
- added D25: D, Diode_THT:D_DO-35_SOD27_P5.08mm_Vertical_AnodeUp, F.Cu at (590.9, 152.5)
- added D26: D, Diode_THT:D_DO-35_SOD27_P5.08mm_Vertical_AnodeUp, F.Cu at (590.9, 156.0)
- added D27: D, Diode_THT:D_DO-35_SOD27_P5.08mm_Vertical_AnodeUp, B.Cu at (135.2, 166.7)
- added D28: D, Diode_THT:D_DO-35_SOD27_P5.08mm_Vertical_AnodeUp, B.Cu at (156.8, 162.2)
- added D29: D, Diode_THT:D_DO-35_SOD27_P5.08mm_Vertical_AnodeUp, B.Cu at (175.9, 157.2)
- added D3: D, Diode_THT:D_DO-35_SOD27_P5.08mm_Vertical_AnodeUp, B.Cu at (175.9, 119.1)
- added D30: D, Diode_THT:D_DO-35_SOD27_P5.08mm_Vertical_AnodeUp, B.Cu at (194.9, 157.9)
- added D31: D, Diode_THT:D_DO-35_SOD27_P5.08mm_Vertical_AnodeUp, B.Cu at (214.0, 162.9)
- added D32: D, Diode_THT:D_DO-35_SOD27_P5.08mm_Vertical_AnodeUp, B.Cu at (233.1, 166.7)
- added D33: D, Diode_THT:D_DO-35_SOD27_P5.08mm_Vertical_AnodeUp, B.Cu at (252.1, 167.0)
- added D34: D, Diode_THT:D_DO-35_SOD27_P5.08mm_Vertical_AnodeUp, F.Cu at (590.9, 184.4)
- added D35: D, Diode_THT:D_DO-35_SOD27_P5.08mm_Vertical_AnodeUp, F.Cu at (601.7, 127.6)
- added D36: D, Diode_THT:D_DO-35_SOD27_P5.08mm_Vertical_AnodeUp, F.Cu at (601.7, 131.2)
- added D37: D, Diode_THT:D_DO-35_SOD27_P5.08mm_Vertical_AnodeUp, F.Cu at (601.7, 134.7)
- added D38: D, Diode_THT:D_DO-35_SOD27_P5.08mm_Vertical_AnodeUp, F.Cu at (601.7, 138.3)
- added D39: D, Diode_THT:D_DO-35_SOD27_P5.08mm_Vertical_AnodeUp, F.Cu at (601.7, 141.8)
- added D4: D, Diode_THT:D_DO-35_SOD27_P5.08mm_Vertical_AnodeUp, B.Cu at (194.9, 119.1)
- added D40: D, Diode_THT:D_DO-35_SOD27_P5.08mm_Vertical_AnodeUp, F.Cu at (601.7, 145.4)
- added D41: D, Diode_THT:D_DO-35_SOD27_P5.08mm_Vertical_AnodeUp, B.Cu at (135.2, 185.7)
- added D42: D, Diode_THT:D_DO-35_SOD27_P5.08mm_Vertical_AnodeUp, B.Cu at (156.8, 183.4)
- added D43: D, Diode_THT:D_DO-35_SOD27_P5.08mm_Vertical_AnodeUp, B.Cu at (175.9, 176.2)
- added D44: D, Diode_THT:D_DO-35_SOD27_P5.08mm_Vertical_AnodeUp, B.Cu at (194.9, 177.2)
- added D45: D, Diode_THT:D_DO-35_SOD27_P5.08mm_Vertical_AnodeUp, B.Cu at (214.0, 181.4)
- added D46: D, Diode_THT:D_DO-35_SOD27_P5.08mm_Vertical_AnodeUp, B.Cu at (233.1, 185.7)
- added D47: D, Diode_THT:D_DO-35_SOD27_P5.08mm_Vertical_AnodeUp, B.Cu at (252.1, 185.7)
- added D48: D, Diode_THT:D_DO-35_SOD27_P5.08mm_Vertical_AnodeUp, F.Cu at (601.7, 173.8)
- added D49: D, Diode_THT:D_DO-35_SOD27_P5.08mm_Vertical_AnodeUp, F.Cu at (601.7, 177.3)
- added D5: D, Diode_THT:D_DO-35_SOD27_P5.08mm_Vertical_AnodeUp, B.Cu at (214.0, 123.8)
- added D50: D, Diode_THT:D_DO-35_SOD27_P5.08mm_Vertical_AnodeUp, F.Cu at (601.7, 180.9)
- added D51: D, Diode_THT:D_DO-35_SOD27_P5.08mm_Vertical_AnodeUp, F.Cu at (601.7, 184.4)
- added D52: D, Diode_THT:D_DO-35_SOD27_P5.08mm_Vertical_AnodeUp, F.Cu at (612.5, 127.6)
- added D53: D, Diode_THT:D_DO-35_SOD27_P5.08mm_Vertical_AnodeUp, F.Cu at (612.5, 131.2)
- added D54: D, Diode_THT:D_DO-35_SOD27_P5.08mm_Vertical_AnodeUp, F.Cu at (612.5, 134.7)
- added D55: D, Diode_THT:D_DO-35_SOD27_P5.08mm_Vertical_AnodeUp, B.Cu at (135.2, 204.8)
- added D56: D, Diode_THT:D_DO-35_SOD27_P5.08mm_Vertical_AnodeUp, B.Cu at (156.8, 204.8)
- added D57: D, Diode_THT:D_DO-35_SOD27_P5.08mm_Vertical_AnodeUp, B.Cu at (175.9, 200.0)
- added D58: D, Diode_THT:D_DO-35_SOD27_P5.08mm_Vertical_AnodeUp, B.Cu at (194.9, 200.0)
- added D59: D, Diode_THT:D_DO-35_SOD27_P5.08mm_Vertical_AnodeUp, B.Cu at (214.0, 204.8)
- added D6: D, Diode_THT:D_DO-35_SOD27_P5.08mm_Vertical_AnodeUp, B.Cu at (233.1, 128.6)
- added D60: D, Diode_THT:D_DO-35_SOD27_P5.08mm_Vertical_AnodeUp, B.Cu at (233.1, 204.8)
- added D61: D, Diode_THT:D_DO-35_SOD27_P5.08mm_Vertical_AnodeUp, B.Cu at (252.1, 204.8)
- added D62: D, Diode_THT:D_DO-35_SOD27_P5.08mm_Vertical_AnodeUp, F.Cu at (612.5, 163.1)
- added D63: D, Diode_THT:D_DO-35_SOD27_P5.08mm_Vertical_AnodeUp, F.Cu at (612.5, 166.7)
- added D64: D, Diode_THT:D_DO-35_SOD27_P5.08mm_Vertical_AnodeUp, F.Cu at (612.5, 170.2)
- added D65: D, Diode_THT:D_DO-35_SOD27_P5.08mm_Vertical_AnodeUp, F.Cu at (612.5, 173.8)
- added D66: D, Diode_THT:D_DO-35_SOD27_P5.08mm_Vertical_AnodeUp, F.Cu at (612.5, 177.3)
- added D67: D, Diode_THT:D_DO-35_SOD27_P5.08mm_Vertical_AnodeUp, F.Cu at (612.5, 180.9)
- added D68: D, Diode_THT:D_DO-35_SOD27_P5.08mm_Vertical_AnodeUp, F.Cu at (612.5, 184.4)
- added D69: D, Diode_THT:D_DO-35_SOD27_P5.08mm_Vertical_AnodeUp, B.Cu at (280.7, 233.7)
- added D7: D, Diode_THT:D_DO-35_SOD27_P5.08mm_Vertical_AnodeUp, B.Cu at (428.3, 123.8)
- added D70: D, Diode_THT:D_DO-35_SOD27_P5.08mm_Vertical_AnodeUp, F.Cu at (623.3, 131.2)
- added D71: D, Diode_THT:D_DO-35_SOD27_P5.08mm_Vertical_AnodeUp, F.Cu at (623.3, 134.7)
- added D72: D, Diode_THT:D_DO-35_SOD27_P5.08mm_Vertical_AnodeUp, F.Cu at (623.3, 138.3)
- added D73: D, Diode_THT:D_DO-35_SOD27_P5.08mm_Vertical_AnodeUp, F.Cu at (623.3, 141.8)
- added D74: D, Diode_THT:D_DO-35_SOD27_P5.08mm_Vertical_AnodeUp, F.Cu at (623.3, 145.4)
- added D75: D, Diode_THT:D_DO-35_SOD27_P5.08mm_Vertical_AnodeUp, B.Cu at (230.5, 252.0)
- added D76: D, Diode_THT:D_DO-35_SOD27_P5.08mm_Vertical_AnodeUp, B.Cu at (246.8, 260.9)
- added D77: D, Diode_THT:D_DO-35_SOD27_P5.08mm_Vertical_AnodeUp, B.Cu at (263.5, 270.2)
- added D78: D, Diode_THT:D_DO-35_SOD27_P5.08mm_Vertical_AnodeUp, F.Cu at (623.3, 159.6)
- added D79: D, Diode_THT:D_DO-35_SOD27_P5.08mm_Vertical_AnodeUp, F.Cu at (623.3, 163.1)
- added D8: D, Diode_THT:D_DO-35_SOD27_P5.08mm_Vertical_AnodeUp, B.Cu at (447.4, 119.1)
- added D80: D, Diode_THT:D_DO-35_SOD27_P5.08mm_Vertical_AnodeUp, F.Cu at (623.3, 166.7)
- added D9: D, Diode_THT:D_DO-35_SOD27_P5.08mm_Vertical_AnodeUp, B.Cu at (466.4, 120.0)
- added J1: Conn_01x04, Connector_PinHeader_2.54mm:PinHeader_1x04_P2.54mm_Vertical, F.Cu at (304.5, 166.4)
- added J2: Conn_01x04, Connector_PinHeader_2.54mm:PinHeader_1x04_P2.54mm_Vertical, F.Cu at (342.6, 176.2)
- added SW1: F1, PCM_Switch_Keyboard_Hotswap_Kailh:SW_Hotswap_Kailh_MX_1.00u, F.Cu at (128.3, 119.1)
- added SW10: F10, PCM_Switch_Keyboard_Hotswap_Kailh:SW_Hotswap_Kailh_MX_1.00u, F.Cu at (475.9, 114.3)
- added SW11: F11, PCM_Switch_Keyboard_Hotswap_Kailh:SW_Hotswap_Kailh_MX_1.00u, F.Cu at (495.0, 119.1)
- added SW12: F12, PCM_Switch_Keyboard_Hotswap_Kailh:SW_Hotswap_Kailh_MX_1.00u, F.Cu at (514.0, 119.1)
- added SW13: Caps, PCM_Switch_Keyboard_Hotswap_Kailh:SW_Hotswap_Kailh_MX_1.50u, F.Cu at (123.5, 138.1)
- added SW14: 1, PCM_Switch_Keyboard_Hotswap_Kailh:SW_Hotswap_Kailh_MX_1.00u, F.Cu at (147.3, 138.1)
- added SW15: 2, PCM_Switch_Keyboard_Hotswap_Kailh:SW_Hotswap_Kailh_MX_1.00u, F.Cu at (166.4, 133.3)
- added SW16: 3, PCM_Switch_Keyboard_Hotswap_Kailh:SW_Hotswap_Kailh_MX_1.00u, F.Cu at (185.4, 128.6)
- added SW17: 4, PCM_Switch_Keyboard_Hotswap_Kailh:SW_Hotswap_Kailh_MX_1.00u, F.Cu at (204.5, 133.3)
- added SW18: 5, PCM_Switch_Keyboard_Hotswap_Kailh:SW_Hotswap_Kailh_MX_1.00u, F.Cu at (223.5, 138.1)
- added SW19: (, PCM_Switch_Keyboard_Hotswap_Kailh:SW_Hotswap_Kailh_MX_1.00u, F.Cu at (242.6, 138.1)
- added SW2: F2, PCM_Switch_Keyboard_Hotswap_Kailh:SW_Hotswap_Kailh_MX_1.00u, F.Cu at (147.3, 119.1)
- added SW20: ), PCM_Switch_Keyboard_Hotswap_Kailh:SW_Hotswap_Kailh_MX_1.00u, F.Cu at (399.7, 138.1)
- added SW21: 6, PCM_Switch_Keyboard_Hotswap_Kailh:SW_Hotswap_Kailh_MX_1.00u, F.Cu at (418.8, 138.1)
- added SW22: 7, PCM_Switch_Keyboard_Hotswap_Kailh:SW_Hotswap_Kailh_MX_1.00u, F.Cu at (437.8, 133.3)
- added SW23: 8, PCM_Switch_Keyboard_Hotswap_Kailh:SW_Hotswap_Kailh_MX_1.00u, F.Cu at (456.9, 128.6)
- added SW24: 9, PCM_Switch_Keyboard_Hotswap_Kailh:SW_Hotswap_Kailh_MX_1.00u, F.Cu at (475.9, 133.3)
- added SW25: 0, PCM_Switch_Keyboard_Hotswap_Kailh:SW_Hotswap_Kailh_MX_1.00u, F.Cu at (495.0, 138.1)
- added SW26: Fn, PCM_Switch_Keyboard_Hotswap_Kailh:SW_Hotswap_Kailh_MX_1.50u, F.Cu at (518.8, 138.1)
- added SW27: Tab, PCM_Switch_Keyboard_Hotswap_Kailh:SW_Hotswap_Kailh_MX_1.50u, F.Cu at (123.5, 157.2)
- added SW28: Q, PCM_Switch_Keyboard_Hotswap_Kailh:SW_Hotswap_Kailh_MX_1.00u, F.Cu at (147.3, 157.2)
- added SW29: W, PCM_Switch_Keyboard_Hotswap_Kailh:SW_Hotswap_Kailh_MX_1.00u, F.Cu at (166.4, 152.4)
- added SW3: F3, PCM_Switch_Keyboard_Hotswap_Kailh:SW_Hotswap_Kailh_MX_1.00u, F.Cu at (166.4, 114.3)
- added SW30: E, PCM_Switch_Keyboard_Hotswap_Kailh:SW_Hotswap_Kailh_MX_1.00u, F.Cu at (185.4, 147.6)
- added SW31: R, PCM_Switch_Keyboard_Hotswap_Kailh:SW_Hotswap_Kailh_MX_1.00u, F.Cu at (204.5, 152.4)
- added SW32: T, PCM_Switch_Keyboard_Hotswap_Kailh:SW_Hotswap_Kailh_MX_1.00u, F.Cu at (223.5, 157.2)
- added SW33: {, PCM_Switch_Keyboard_Hotswap_Kailh:SW_Hotswap_Kailh_MX_1.00u, F.Cu at (242.6, 157.2)
- added SW34: }, PCM_Switch_Keyboard_Hotswap_Kailh:SW_Hotswap_Kailh_MX_1.00u, F.Cu at (399.7, 157.2)
- added SW35: Y, PCM_Switch_Keyboard_Hotswap_Kailh:SW_Hotswap_Kailh_MX_1.00u, F.Cu at (418.8, 157.2)
- added SW36: U, PCM_Switch_Keyboard_Hotswap_Kailh:SW_Hotswap_Kailh_MX_1.00u, F.Cu at (437.8, 152.4)
- added SW37: I, PCM_Switch_Keyboard_Hotswap_Kailh:SW_Hotswap_Kailh_MX_1.00u, F.Cu at (456.9, 147.6)
- added SW38: O, PCM_Switch_Keyboard_Hotswap_Kailh:SW_Hotswap_Kailh_MX_1.00u, F.Cu at (475.9, 152.4)
- added SW39: P, PCM_Switch_Keyboard_Hotswap_Kailh:SW_Hotswap_Kailh_MX_1.00u, F.Cu at (495.0, 157.2)
- added SW4: F4, PCM_Switch_Keyboard_Hotswap_Kailh:SW_Hotswap_Kailh_MX_1.00u, F.Cu at (185.4, 109.5)
- added SW40: =, PCM_Switch_Keyboard_Hotswap_Kailh:SW_Hotswap_Kailh_MX_1.50u, F.Cu at (518.8, 157.2)
- added SW41: Esc, PCM_Switch_Keyboard_Hotswap_Kailh:SW_Hotswap_Kailh_MX_1.50u, F.Cu at (123.5, 176.2)
- added SW42: A, PCM_Switch_Keyboard_Hotswap_Kailh:SW_Hotswap_Kailh_MX_1.00u, F.Cu at (147.3, 176.2)
- added SW43: S, PCM_Switch_Keyboard_Hotswap_Kailh:SW_Hotswap_Kailh_MX_1.00u, F.Cu at (166.4, 171.4)
- added SW44: D, PCM_Switch_Keyboard_Hotswap_Kailh:SW_Hotswap_Kailh_MX_1.00u, F.Cu at (185.4, 166.7)
- added SW45: F, PCM_Switch_Keyboard_Hotswap_Kailh:SW_Hotswap_Kailh_MX_1.00u, F.Cu at (204.5, 171.4)
- added SW46: G, PCM_Switch_Keyboard_Hotswap_Kailh:SW_Hotswap_Kailh_MX_1.00u, F.Cu at (223.5, 176.2)
- added SW47: [, PCM_Switch_Keyboard_Hotswap_Kailh:SW_Hotswap_Kailh_MX_1.00u, F.Cu at (242.6, 176.2)
- added SW48: ], PCM_Switch_Keyboard_Hotswap_Kailh:SW_Hotswap_Kailh_MX_1.00u, F.Cu at (399.7, 176.2)
- added SW49: H, PCM_Switch_Keyboard_Hotswap_Kailh:SW_Hotswap_Kailh_MX_1.00u, F.Cu at (418.8, 176.2)
- added SW5: F5, PCM_Switch_Keyboard_Hotswap_Kailh:SW_Hotswap_Kailh_MX_1.00u, F.Cu at (204.5, 114.3)
- added SW50: J, PCM_Switch_Keyboard_Hotswap_Kailh:SW_Hotswap_Kailh_MX_1.00u, F.Cu at (437.8, 171.4)
- added SW51: K, PCM_Switch_Keyboard_Hotswap_Kailh:SW_Hotswap_Kailh_MX_1.00u, F.Cu at (456.9, 166.7)
- added SW52: L, PCM_Switch_Keyboard_Hotswap_Kailh:SW_Hotswap_Kailh_MX_1.00u, F.Cu at (475.9, 171.4)
- added SW53: ;, PCM_Switch_Keyboard_Hotswap_Kailh:SW_Hotswap_Kailh_MX_1.00u, F.Cu at (495.0, 176.2)
- added SW54: -, PCM_Switch_Keyboard_Hotswap_Kailh:SW_Hotswap_Kailh_MX_1.50u, F.Cu at (518.8, 176.2)
- added SW55: Shift, PCM_Switch_Keyboard_Hotswap_Kailh:SW_Hotswap_Kailh_MX_1.50u, F.Cu at (123.5, 195.3)
- added SW56: Z, PCM_Switch_Keyboard_Hotswap_Kailh:SW_Hotswap_Kailh_MX_1.00u, F.Cu at (147.3, 195.3)
- added SW57: X, PCM_Switch_Keyboard_Hotswap_Kailh:SW_Hotswap_Kailh_MX_1.00u, F.Cu at (166.4, 190.5)
- added SW58: C, PCM_Switch_Keyboard_Hotswap_Kailh:SW_Hotswap_Kailh_MX_1.00u, F.Cu at (185.4, 185.7)
- added SW59: V, PCM_Switch_Keyboard_Hotswap_Kailh:SW_Hotswap_Kailh_MX_1.00u, F.Cu at (204.5, 190.5)
- added SW6: F6, PCM_Switch_Keyboard_Hotswap_Kailh:SW_Hotswap_Kailh_MX_1.00u, F.Cu at (223.5, 119.1)
- added SW60: B, PCM_Switch_Keyboard_Hotswap_Kailh:SW_Hotswap_Kailh_MX_1.00u, F.Cu at (223.5, 195.3)
- added SW61: ', PCM_Switch_Keyboard_Hotswap_Kailh:SW_Hotswap_Kailh_MX_1.00u, F.Cu at (242.6, 195.3)
- added SW62: ", PCM_Switch_Keyboard_Hotswap_Kailh:SW_Hotswap_Kailh_MX_1.00u, F.Cu at (399.7, 195.3)
- added SW63: N, PCM_Switch_Keyboard_Hotswap_Kailh:SW_Hotswap_Kailh_MX_1.00u, F.Cu at (418.8, 195.3)
- added SW64: M, PCM_Switch_Keyboard_Hotswap_Kailh:SW_Hotswap_Kailh_MX_1.00u, F.Cu at (437.8, 190.5)
- added SW65: ,, PCM_Switch_Keyboard_Hotswap_Kailh:SW_Hotswap_Kailh_MX_1.00u, F.Cu at (456.9, 185.7)
- added SW66: ., PCM_Switch_Keyboard_Hotswap_Kailh:SW_Hotswap_Kailh_MX_1.00u, F.Cu at (475.9, 190.5)
- added SW67: "/", PCM_Switch_Keyboard_Hotswap_Kailh:SW_Hotswap_Kailh_MX_1.00u, F.Cu at (495.0, 195.3)
- added SW68: RShift, PCM_Switch_Keyboard_Hotswap_Kailh:SW_Hotswap_Kailh_MX_1.50u, F.Cu at (518.8, 195.3)
- added SW69: Space, PCM_Switch_Keyboard_Hotswap_Kailh:SW_Hotswap_Kailh_MX_2.00u, F.Cu at (267.9, 224.3)
- added SW7: F7, PCM_Switch_Keyboard_Hotswap_Kailh:SW_Hotswap_Kailh_MX_1.00u, F.Cu at (418.8, 119.1)
- added SW71: Left, PCM_Switch_Keyboard_Hotswap_Kailh:SW_Hotswap_Kailh_MX_1.00u, F.Cu at (437.8, 209.6)
- added SW72: Down, PCM_Switch_Keyboard_Hotswap_Kailh:SW_Hotswap_Kailh_MX_1.00u, F.Cu at (456.9, 204.8)
- added SW73: Up, PCM_Switch_Keyboard_Hotswap_Kailh:SW_Hotswap_Kailh_MX_1.00u, F.Cu at (475.9, 209.6)
- added SW74: Right, PCM_Switch_Keyboard_Hotswap_Kailh:SW_Hotswap_Kailh_MX_1.00u, F.Cu at (495.0, 214.3)
- added SW75: Ctrl, PCM_Switch_Keyboard_Hotswap_Kailh:SW_Hotswap_Kailh_MX_2.00u_90deg, F.Cu at (228.9, 234.8)
- added SW76: Linux, PCM_Switch_Keyboard_Hotswap_Kailh:SW_Hotswap_Kailh_MX_2.00u_90deg, F.Cu at (245.3, 244.4)
- added SW77: alt, PCM_Switch_Keyboard_Hotswap_Kailh:SW_Hotswap_Kailh_MX_2.00u_90deg, F.Cu at (261.8, 253.8)
- added SW8: F8, PCM_Switch_Keyboard_Hotswap_Kailh:SW_Hotswap_Kailh_MX_1.00u, F.Cu at (437.8, 114.3)
- added SW9: F9, PCM_Switch_Keyboard_Hotswap_Kailh:SW_Hotswap_Kailh_MX_1.00u, F.Cu at (456.9, 109.5)
Routing:
- net L_COL6: track 0.00 -> 374.2 mm
- net L_COL0: track 0.00 -> 271.7 mm
- net L_COL1: track 0.00 -> 259.0 mm
- net L_COL4: track 0.00 -> 253.9 mm
- net L_COL2: track 0.00 -> 242.5 mm
- net L_COL5: track 0.00 -> 229.0 mm
- net L_COL3: track 0.00 -> 218.8 mm
- net L_ROW0: track 0.00 -> 175.1 mm
- net L_ROW1: track 0.00 -> 160.3 mm
- net L_ROW3: track 0.00 -> 148.0 mm
- net L_ROW2: track 0.00 -> 145.3 mm
- net L_ROW6: track 0.00 -> 130.0 mm
- net R_ROW0: track 0.00 -> 101.3 mm
- net R_COL1: track 0.00 -> 95.3 mm
- net R_COL3: track 0.00 -> 95.2 mm
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
Commit message: refactor(argv-split): update keyboard and PCB layout
Parts:
- removed D71, D72, D73, D74: D, Diode_THT:D_DO-35_SOD27_P5.08mm_Vertical_AnodeUp
- removed SW71: Left, PCM_Switch_Keyboard_Hotswap_Kailh:SW_Hotswap_Kailh_MX_1.00u
- removed SW72: Down, PCM_Switch_Keyboard_Hotswap_Kailh:SW_Hotswap_Kailh_MX_1.00u
- removed SW73: Up, PCM_Switch_Keyboard_Hotswap_Kailh:SW_Hotswap_Kailh_MX_1.00u
- removed SW74: Right, PCM_Switch_Keyboard_Hotswap_Kailh:SW_Hotswap_Kailh_MX_1.00u
- added SW70: Backspace, PCM_Switch_Keyboard_Hotswap_Kailh:SW_Hotswap_Kailh_MX_2.00u, F.Cu at (184.1, 168.2)
- added SW78: Return, PCM_Switch_Keyboard_Hotswap_Kailh:SW_Hotswap_Kailh_MX_2.00u_90deg, F.Cu at (184.1, 230.4)
- added SW79: Linux, PCM_Switch_Keyboard_Hotswap_Kailh:SW_Hotswap_Kailh_MX_2.00u_90deg, F.Cu at (184.1, 246.0)
- added SW80: Ctrl, PCM_Switch_Keyboard_Hotswap_Kailh:SW_Hotswap_Kailh_MX_2.00u_90deg, F.Cu at (184.1, 261.5)
- A2, D1, D10, D11, D12, D13, D14, D15, D16, D17, D18, D19, D2, D27, D28, D29, D3, D30, D31, D32, D33, D4, D41, D42, D43, D44, D45, D46, D47, D5, D55, D56, D57, D58, D59, D6, D60, D61, D69, D7, D75, D76, D77, D8, D9: moved to F.Cu
- moved SW11 440.1 mm to (84.2, 277.1)
- moved SW10 418.4 mm to (84.2, 261.5)
- moved SW12 413.2 mm to (100.9, 121.6)
- moved D52 407.9 mm to (219.3, 236.2)
- moved SW26 402.4 mm to (117.5, 168.2)
- moved D39 402.1 mm to (210.8, 236.2)
- moved D38 402.1 mm to (210.8, 232.4)
- moved D37 402.0 mm to (210.8, 228.6)
- moved D36 402.0 mm to (210.8, 224.9)
- moved D35 401.9 mm to (210.8, 221.1)
- moved D26 396.9 mm to (202.3, 236.2)
- moved SW9 396.8 mm to (84.2, 246.0)
- moved D25 396.8 mm to (202.3, 232.4)
- moved D24 396.8 mm to (202.3, 228.6)
- moved D23 396.7 mm to (202.3, 224.9)
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Connections:
- A1 pad 15: L_COL6 -> L_ROW4
- A1 pad 26: /GPIO20 -> /L_GPIO20
- A1 pad 27: /GPIO21 -> /L_GPIO21
- A1 pad 33: unconnected-(A1-AGND-Pad33) -> /GND
- A2 pad 1: unconnected-(A2-GPIO0-Pad1) -> R_COL0
- A2 pad 10: unconnected-(A2-GPIO7-Pad10) -> R_ROW0
- A2 pad 11: unconnected-(A2-GPIO8-Pad11) -> R_ROW1
- A2 pad 12: unconnected-(A2-GPIO9-Pad12) -> R_ROW2
- A2 pad 14: unconnected-(A2-GPIO10-Pad14) -> R_ROW3
- A2 pad 15: unconnected-(A2-GPIO11-Pad15) -> R_ROW4
- A2 pad 16: unconnected-(A2-GPIO12-Pad16) -> R_ROW5
- A2 pad 17: unconnected-(A2-GPIO13-Pad17) -> R_ROW6
- A2 pad 2: unconnected-(A2-GPIO1-Pad2) -> R_COL1
- A2 pad 26: /GPIO20 -> /R_GPIO20
- A2 pad 27: /GPIO21 -> /R_GPIO21
- A2 pad 33: unconnected-(A2-AGND-Pad33) -> /GND
- A2 pad 4: unconnected-(A2-GPIO2-Pad4) -> R_COL2
- A2 pad 5: unconnected-(A2-GPIO3-Pad5) -> R_COL3
- A2 pad 6: unconnected-(A2-GPIO4-Pad6) -> R_COL4
- A2 pad 7: unconnected-(A2-GPIO5-Pad7) -> R_COL5
- A2 pad 9: unconnected-(A2-GPIO6-Pad9) -> R_COL6
- D55 pad 1: L_COL6 -> L_ROW4
- D56 pad 1: L_COL6 -> L_ROW4
- D57 pad 1: L_COL6 -> L_ROW4
- D58 pad 1: L_COL6 -> L_ROW4
- D59 pad 1: L_COL6 -> L_ROW4
- D60 pad 1: L_COL6 -> L_ROW4
- D61 pad 1: L_COL6 -> L_ROW4
- D70 pad 1: R_COL6 -> R_ROW5
- J1 pad 2: /GPIO21 -> /L_GPIO21
- J1 pad 3: /GPIO20 -> /L_GPIO20
- J2 pad 2: /GPIO20 -> /R_GPIO20
- J2 pad 3: /GPIO21 -> /R_GPIO21
Routing:
- net L_COL6: track 374.2 -> 0.00 mm
- net L_COL0: track 271.7 -> 0.00 mm
- net L_COL1: track 259.0 -> 0.00 mm
- net L_COL4: track 253.9 -> 0.00 mm
- net L_COL2: track 242.5 -> 0.00 mm
- net L_COL5: track 229.0 -> 0.00 mm
- net L_COL3: track 218.8 -> 0.00 mm
- net L_ROW0: track 175.1 -> 0.00 mm
- net L_ROW1: track 160.3 -> 0.00 mm
- net L_ROW3: track 148.0 -> 0.00 mm
- net L_ROW2: track 145.3 -> 0.00 mm
- net L_ROW6: track 130.0 -> 0.00 mm
- net R_ROW0: track 101.3 -> 0.00 mm
- net R_COL1: track 95.3 -> 0.00 mm
- net R_COL3: track 95.2 -> 0.00 mm
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
Commit message: feat: new layout
Parts:
- removed D77, D78, D79, D80: D, Diode_THT:D_DO-35_SOD27_P5.08mm_Vertical_AnodeUp
- removed J1, J2: Conn_01x04, Connector_PinHeader_2.54mm:PinHeader_1x04_P2.54mm_Vertical
- removed SW77: alt, PCM_Switch_Keyboard_Hotswap_Kailh:SW_Hotswap_Kailh_MX_2.00u_90deg
- removed SW78: Return, PCM_Switch_Keyboard_Hotswap_Kailh:SW_Hotswap_Kailh_MX_2.00u_90deg
- removed SW79: Linux, PCM_Switch_Keyboard_Hotswap_Kailh:SW_Hotswap_Kailh_MX_2.00u_90deg
- removed SW80: Ctrl, PCM_Switch_Keyboard_Hotswap_Kailh:SW_Hotswap_Kailh_MX_2.00u_90deg
- added D71: D, Diode_THT:D_DO-35_SOD27_P7.62mm_Horizontal, B.Cu at (209.8, 253.9)
- added D72: D, Diode_THT:D_DO-35_SOD27_P7.62mm_Horizontal, B.Cu at (226.3, 263.5)
- added D73: D, Diode_THT:D_DO-35_SOD27_P7.62mm_Horizontal, B.Cu at (242.8, 273.0)
- added D74: D, Diode_THT:D_DO-35_SOD27_P7.62mm_Horizontal, B.Cu at (392.1, 263.5)
- added J3: AudioJack4, Connector_Audio:Jack_3.5mm_PJ320E_Horizontal, F.Cu at (286.2, 131.1)
- added J4: AudioJack4, Connector_Audio:Jack_3.5mm_PJ320E_Horizontal, F.Cu at (331.8, 135.7)
- added SW71: Ctrl, PCM_Switch_Keyboard_Hotswap_Kailh:SW_Hotswap_Kailh_MX_2.00u_90deg, F.Cu at (211.1, 232.7)
- added SW72: Linux, PCM_Switch_Keyboard_Hotswap_Kailh:SW_Hotswap_Kailh_MX_2.00u_90deg, F.Cu at (227.6, 242.2)
- added SW73: alt, PCM_Switch_Keyboard_Hotswap_Kailh:SW_Hotswap_Kailh_MX_2.00u_90deg, F.Cu at (244.1, 251.7)
- added SW74: Return, PCM_Switch_Keyboard_Hotswap_Kailh:SW_Hotswap_Kailh_MX_2.00u_90deg, F.Cu at (374.4, 251.8)
- A2: moved to B.Cu
- D1, D10, D11, D12, D13, D14, D15, D16, D17, D18, D19, D2, D20, D21, D22, D23, D24, D25, D26, D27, D28, D29, D3, D30, D31, D32, D33, D34, D35, D36, D37, D38, D39, D4, D40, D41, D42, D43, D44, D45, D46, D47, D48, D49, D5, D50, D51, D52, D53, D54, D55, D56, D57, D58, D59, D6, D60, D61, D62, D63, D64, D65, D66, D67, D68, D69, D7, D70, D75, D76, D8, D9: footprint Diode_THT:D_DO-35_SOD27_P5.08mm_Vertical_AnodeUp -> Diode_THT:D_DO-35_SOD27_P7.62mm_Horizontal; moved to B.Cu
- SW75: value Ctrl -> Linux
- SW76: value Linux -> Ctrl
- moved SW11 417.9 mm to (471.2, 119.1)
- moved SW26 397.7 mm to (514.0, 138.1)
- moved SW10 394.5 mm to (452.1, 119.1)
- moved SW12 389.4 mm to (490.2, 119.1)
- moved SW40 384.2 mm to (514.0, 157.2)
- moved SW54 373.1 mm to (514.0, 176.2)
- moved SW25 373.0 mm to (490.2, 138.1)
- moved SW9 371.2 mm to (433.1, 119.1)
- moved SW22 360.1 mm to (433.1, 138.1)
- moved SW39 358.6 mm to (490.2, 157.2)
- moved SW24 353.7 mm to (471.2, 138.1)
- moved SW8 348.1 mm to (414.0, 119.1)
- moved SW53 346.5 mm to (490.2, 176.2)
- moved SW38 338.1 mm to (471.2, 157.2)
- moved SW21 336.6 mm to (414.0, 138.1)
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Connections:
- A1 pad 39: unconnected-(A1-VSYS-Pad39)_1 -> /R_VSYS
- A1 pad 40: /VBUS -> unconnected-(A1-VBUS-Pad40)
- A2 pad 39: /VSYS -> /L_VSYS
- D75 pad 1: L_ROW6 -> R_ROW6
- D76 pad 1: L_ROW6 -> R_ROW6
- SW1 pad 1: L_COL0 -> L_COL1
- SW10 pad 1: R_COL2 -> R_COL3
- SW11 pad 1: R_COL1 -> R_COL2
- SW12 pad 1: R_COL0 -> R_COL1
- SW2 pad 1: L_COL1 -> L_COL2
- SW3 pad 1: L_COL2 -> L_COL3
- SW4 pad 1: L_COL3 -> L_COL4
- SW5 pad 1: L_COL4 -> L_COL5
- SW6 pad 1: L_COL5 -> L_COL6
- SW7 pad 1: R_COL5 -> R_COL6
- SW75 pad 1: L_COL4 -> R_COL5
- SW76 pad 1: L_COL5 -> R_COL4
- SW8 pad 1: R_COL4 -> R_COL5
- SW9 pad 1: R_COL3 -> R_COL4
Routing:
- net L_COL0: track 0.00 -> 238.7 mm
- net R_COL0: track 0.00 -> 231.8 mm
- net R_COL4: track 0.00 -> 228.4 mm
- net R_COL1: track 0.00 -> 213.5 mm
- net R_COL5: track 0.00 -> 209.4 mm
- net R_ROW4: track 0.00 -> 207.2 mm
- net L_COL1: track 0.00 -> 206.0 mm
- net R_COL6: track 0.00 -> 204.3 mm
- net R_COL2: track 0.00 -> 198.4 mm
- net L_COL4: track 0.00 -> 196.4 mm
- net R_ROW3: track 0.00 -> 191.0 mm
- net L_COL2: track 0.00 -> 190.8 mm
- net L_COL6: track 0.00 -> 188.7 mm
- net L_COL5: track 0.00 -> 186.6 mm
- net L_ROW4: track 0.00 -> 183.0 mm
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- added copper zone on B.Cu, net /GND
- added copper zone on F.Cu, net /GND
Other:
- board outline added: 447 x 185.7 mm
