File: argv_split/argv_split_kicad/argv_split_kicad.kicad_pcb (KiCad board)
At the start: 2 copper layers, 447 x 185.7 mm, 156 parts, among them J3 AudioJack4, J4 AudioJack4, SW1 F1, SW10 F10, SW11 F11, SW12 F12, SW13 Caps, SW14 1, SW15 2, SW16 3, SW17 4, SW18 5, SW19 (, SW2 F2, SW20 ), SW21 6, SW22 7, SW23 8, SW24 9, SW25 0, SW26 Fn, SW27 Tab, SW28 Q, SW29 W, SW3 F3, SW30 E, SW31 R, SW32 T, SW33 {, SW34 }, SW35 Y, SW36 U, SW37 I, SW38 O, SW39 P, SW4 F4, SW40 =, SW41 Esc, SW42 A, SW43 S, SW44 D, SW45 F, SW46 G, SW47 [, SW48 ], SW49 H, SW5 F5, SW50 J, SW51 K, SW52 L, SW53 ;, SW54 -, SW55 Shift, SW56 Z, SW57 X, SW58 C, SW59 V, SW6 F6, SW60 B, SW61 ', SW62 ", SW63 N, SW64 M, SW65 ,, SW66 ., SW67 "/", SW68 RShift, SW69 Space, SW7 F7, SW70 Backspace, SW71 Ctrl, SW72 Linux, SW73 alt, SW74 Return, SW75 Linux, SW76 Ctrl, SW8 F8, SW9 F9

Commit message: fix(split): pcb layout
Parts:
- added REF**: MountingHole_2.1mm, MountingHole:MountingHole_2.1mm, F.Cu at (252.1, 166.7)
- added REF**: MountingHole_2.1mm, MountingHole:MountingHole_2.1mm, F.Cu at (114.0, 119.1)
- added REF**: MountingHole_2.1mm, MountingHole:MountingHole_2.1mm, F.Cu at (433.1, 104.8)
- added REF**: MountingHole_2.1mm, MountingHole:MountingHole_2.1mm, F.Cu at (485.5, 104.8)
- added REF**: MountingHole_2.1mm, MountingHole:MountingHole_2.1mm, F.Cu at (242.6, 128.6)
- added REF**: MountingHole_2.1mm, MountingHole:MountingHole_2.1mm, F.Cu at (228.3, 214.3)
- added REF**: MountingHole_2.1mm, MountingHole:MountingHole_2.1mm, F.Cu at (285.4, 123.8)
- added REF**: MountingHole_2.1mm, MountingHole:MountingHole_2.1mm, F.Cu at (237.8, 190.5)
- added REF**: MountingHole_2.1mm, MountingHole:MountingHole_2.1mm, F.Cu at (204.5, 214.3)
- added REF**: MountingHole_2.1mm, MountingHole:MountingHole_2.1mm, F.Cu at (414.0, 214.3)
- added REF**: MountingHole_2.1mm, MountingHole:MountingHole_2.1mm, F.Cu at (371.2, 195.3)
- added REF**: MountingHole_2.1mm, MountingHole:MountingHole_2.1mm, F.Cu at (366.4, 166.7)
- added REF**: MountingHole_2.1mm, MountingHole:MountingHole_2.1mm, F.Cu at (333.1, 119.1)
- added REF**: MountingHole_2.1mm, MountingHole:MountingHole_2.1mm, F.Cu at (390.2, 209.6)

Commit message: feat(split): done pcb design
Parts:
- removed REF** (x14): MountingHole_2.1mm, MountingHole:MountingHole_2.1mm
Routing:
- net L_COL3: track 171.6 -> 190.7 mm
- net L_COL6: track 188.7 -> 207.8 mm
- net L_COL5: track 186.6 -> 205.6 mm
- net L_COL4: track 196.4 -> 215.5 mm
- net L_COL2: track 190.8 -> 209.8 mm
- net L_COL1: track 206.0 -> 225.0 mm
- net /GND: track 23.2 -> 39.0 mm
- net Net-(D55-A): track 0.00 -> 11.3 mm
- net Net-(D51-A): track 0.00 -> 8.51 mm
