File: argv_split/argv-split-pcb/argv-split.kicad_pcb (KiCad board)
At the start: 2 copper layers, 434.1 x 180.4 mm, 160 parts, among them SW1 SW_Push, SW10 SW_Push, SW11 SW_Push, SW12 SW_Push, SW13 SW_Push, SW14 SW_Push, SW15 SW_Push, SW16 SW_Push, SW17 SW_Push, SW18 SW_Push, SW19 SW_Push, SW2 SW_Push, SW20 SW_Push, SW21 SW_Push, SW22 SW_Push, SW23 SW_Push, SW24 SW_Push, SW25 SW_Push, SW26 SW_Push, SW27 SW_Push, SW28 SW_Push, SW29 SW_Push, SW3 SW_Push, SW30 SW_Push, SW31 SW_Push, SW32 SW_Push, SW33 SW_Push, SW34 SW_Push, SW35 SW_Push, SW36 SW_Push, SW37 SW_Push, SW38 SW_Push, SW39 SW_Push, SW4 SW_Push, SW40 SW_Push, SW41 SW_Push, SW42 SW_Push, SW43 SW_Push, SW44 SW_Push, SW45 SW_Push, SW46 SW_Push, SW47 SW_Push, SW48 SW_Push, SW49 SW_Push, SW5 SW_Push, SW50 SW_Push, SW51 SW_Push, SW52 SW_Push, SW53 SW_Push, SW54 SW_Push, SW55 SW_Push, SW56 SW_Push, SW57 SW_Push, SW58 SW_Push, SW59 SW_Push, SW6 SW_Push, SW60 SW_Push, SW61 SW_Push, SW62 SW_Push, SW63 SW_Push, SW64 SW_Push, SW65 SW_Push, SW66 SW_Push, SW67 SW_Push, SW68 SW_Push, SW69 SW_Push, SW7 SW_Push, SW70 SW_Push, SW71 SW_Push, SW72 SW_Push, SW73 SW_Push, SW74 SW_Push, SW75 SW_Push, SW76 SW_Push, SW8 SW_Push, SW9 SW_Push

Commit message: feat: layout pcb
Parts:
- D1, D10, D11, D12, D13, D14, D15, D16, D17, D18, D19, D2, D20, D21, D22, D23, D24, D25, D26, D27, D28, D29, D3, D30, D31, D32, D33, D34, D35, D36, D37, D38, D39, D4, D40, D41, D42, D43, D44, D45, D46, D47, D48, D49, D5, D50, D51, D52, D53, D54, D55, D56, D57, D58, D59, D6, D60, D61, D62, D63, D64, D65, D66, D67, D68, D69, D7, D70, D71, D72, D73, D74, D75, D76, D8, D9: footprint Diode_SMD:D_SOD-123 -> Diode_THT:D_DO-35_SOD27_P7.62mm_Horizontal
- moved D36 13.6 mm to (134.1, 119.3)
- moved D76 6.73 mm to (254.3, 129.3)
- moved D53 6.73 mm to (276.4, 47.0)
- moved D54 6.73 mm to (295.5, 47.0)
- moved D55 6.73 mm to (314.6, 47.0)
- moved D56 6.73 mm to (333.6, 47.0)
- moved D60 6.73 mm to (276.4, 66.0)
- moved D61 6.73 mm to (295.5, 66.0)
- moved D62 6.73 mm to (314.6, 66.0)
- moved D63 6.73 mm to (333.6, 66.0)
- moved D40 6.73 mm to (276.4, 8.85)
- moved D41 6.73 mm to (295.5, 8.85)
- moved D42 6.73 mm to (314.6, 8.85)
- moved D43 6.73 mm to (333.6, 8.85)
- moved D46 6.73 mm to (276.4, 27.9)
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Routing:
- net COL6: track 0.00 -> 123.0 mm
- net ROW3: track 0.00 -> 119.1 mm
- net ROW1: track 0.00 -> 119.1 mm
- net ROW4: track 0.00 -> 119.1 mm
- net ROW2: track 0.00 -> 119.1 mm
- net COL5: track 0.00 -> 114.6 mm
- net ROW0: track 0.00 -> 95.2 mm, vias 0 -> 1
- net COL4: track 0.00 -> 76.2 mm
- net COL3: track 0.00 -> 76.2 mm
- net COL2: track 0.00 -> 76.2 mm
- net COL1: track 0.00 -> 76.2 mm
- net COL0: track 0.00 -> 57.1 mm
- net ROW5: track 0.00 -> 52.1 mm
- net COL7: track 0.00 -> 33.3 mm
- net ROW6: track 0.00 -> 20.7 mm
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Other:
- board outline removed

Commit message: feat(split): routing
Parts:
- added A1: RaspberryPi_Pico, Module:RaspberryPi_Pico_Common_Unspecified, F.Cu at (129.0, 16.9)
- added A2: RaspberryPi_Pico, Module:RaspberryPi_Pico_Common_Unspecified, B.Cu at (218.5, 16.7)
- moved D73 12.3 mm to (241.0, 101.2)
- moved D76 3.76 mm to (255.5, 125.7)
- moved D74 3.27 mm to (272.4, 116.9)
- moved D75 3.26 mm to (238.8, 135.7)
Routing:
- net COL0: track 57.1 -> 245.4 mm
- net ROW6: track 20.7 -> 176.6 mm
- net COL1: track 76.2 -> 231.3 mm
- net COL2: track 76.2 -> 214.8 mm
- net COL9: track 0.00 -> 132.2 mm, vias 0 -> 1
- net ROW5: track 52.1 -> 179.0 mm
- net COL3: track 76.2 -> 199.2 mm
- net COL10: track 0.00 -> 120.9 mm
- net ROW9: track 0.00 -> 119.1 mm
- net ROW8: track 0.00 -> 119.1 mm
- net ROW11: track 0.00 -> 119.1 mm, vias 0 -> 1
- net ROW10: track 0.00 -> 119.1 mm
- net COL4: track 76.2 -> 182.0 mm
- net ROW7: track 0.00 -> 95.2 mm
- net ROW4: track 119.1 -> 209.2 mm
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