File: argv_split/argv-split-pcb/keyboard.kicad_pcb (KiCad board)
At the start: 2 copper layers, 184 x 152 mm, 78 parts, among them J1 BREAKOUT_4PIN, SW1 SW_Push, SW10 SW_Push, SW11 SW_Push, SW12 SW_Push, SW13 SW_Push, SW14 SW_Push, SW15 SW_Push, SW16 SW_Push, SW17 SW_Push, SW18 SW_Push, SW19 SW_Push, SW2 SW_Push, SW20 SW_Push, SW21 SW_Push, SW22 SW_Push, SW23 SW_Push, SW24 SW_Push, SW25 SW_Push, SW26 SW_Push, SW27 SW_Push, SW28 SW_Push, SW29 SW_Push, SW3 SW_Push, SW4 SW_Push, SW5 SW_Push, SW6 SW_Push, SW62 SW_Push, SW63 SW_Push, SW64 SW_Push, SW7 SW_Push, SW8 SW_Push, SW9 SW_Push, U1 RaspberryPi_Pico

Commit message: untested: learning from ai slop
Parts:
- added H7: MountingHole_2.1mm, MountingHole:MountingHole_2.1mm, F.Cu at (209.6, 121.9)
- added H7: MountingHole_2.1mm, MountingHole:MountingHole_2.1mm, F.Cu at (152.2, 122.2)
- U1: footprint Module:RaspberryPi_Pico_Common_THT -> ARGV:RaspberryPi_Pico_Case_THT
- moved H2 152.6 mm to (255.7, 81.2)
- moved H5 151.4 mm to (203.2, 163.8)
- moved H3 151.3 mm to (285.3, 81.0)
- moved D17 150.6 mm to (171.0, 138.1)
- moved D20 150.6 mm to (228.1, 138.1)
- moved D1 150.6 mm to (128.1, 100.0)
- moved D10 150.6 mm to (171.0, 119.1)
- moved D13 150.6 mm to (228.1, 119.1)
- moved D14 150.6 mm to (247.2, 119.1)
- moved D15 150.6 mm to (128.1, 138.1)
- moved D16 150.6 mm to (151.9, 138.1)
- moved D18 150.6 mm to (190.0, 138.1)
- moved D19 150.6 mm to (209.1, 138.1)
- moved D2 150.6 mm to (151.9, 100.0)
- moved D21 150.6 mm to (247.2, 138.1)
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- renumbered REF** to H1, REF** to H2, REF** to H3, REF** to H4, REF** to H5, REF** to H6, REF** to H7, REF** to H8
Routing:
- net L_GND: track 60.3 -> 129.4 mm, vias 0 -> 1
- net L_VSYS: track 0.00 -> 66.2 mm, vias 0 -> 1
- net COL1: track 184.3 -> 200.3 mm
- net Net-(D63-A): track 19.2 -> 6.58 mm
- net ROW9: track 143.0 -> 153.8 mm, vias 1 -> 0
- net ROW1: track 146.7 -> 156.5 mm
- net COL7: track 70.0 -> 78.2 mm
- net ROW2: track 163.2 -> 171.2 mm
- net COL4: track 130.4 -> 126.3 mm
- net ROW0: track 135.9 -> 139.2 mm
- net COL0: track 208.9 -> 211.7 mm
- net COL3: track 150.1 -> 148.1 mm
- net ROW3: track 231.8 -> 233.7 mm, vias 1 -> 0
- net COL2: track 164.7 -> 165.7 mm
- net COL6: track 134.4 -> 133.8 mm
- added copper zone on B.Cu, net L_GND
- added copper zone on F.Cu, net L_GND
Other:
- board size 184 x 152 mm -> 184.4 x 152 mm
- board text removed: "5 mm MIN EDGE PADDING"
