File: argv_split/argv-split-pcb/keyboard.kicad_sch (KiCad schematic)
At the start: 140 parts, among them J1 BREAKOUT_4PIN, J2 BREAKOUT_4PIN, SW1 SW_Push, SW10 SW_Push, SW11 SW_Push, SW12 SW_Push, SW13 SW_Push, SW14 SW_Push, SW15 SW_Push, SW16 SW_Push, SW17 SW_Push, SW18 SW_Push, SW19 SW_Push, SW2 SW_Push, SW20 SW_Push, SW21 SW_Push, SW22 SW_Push, SW23 SW_Push, SW24 SW_Push, SW25 SW_Push, SW26 SW_Push, SW27 SW_Push, SW28 SW_Push, SW29 SW_Push, SW3 SW_Push, SW30 SW_Push, SW31 SW_Push, SW32 SW_Push, SW33 SW_Push, SW34 SW_Push, SW35 SW_Push, SW36 SW_Push, SW37 SW_Push, SW38 SW_Push, SW39 SW_Push, SW4 SW_Push, SW40 SW_Push, SW41 SW_Push, SW42 SW_Push, SW43 SW_Push, SW44 SW_Push, SW45 SW_Push, SW46 SW_Push, SW47 SW_Push, SW48 SW_Push, SW49 SW_Push, SW5 SW_Push, SW50 SW_Push, SW51 SW_Push, SW52 SW_Push, SW53 SW_Push, SW54 SW_Push, SW55 SW_Push, SW56 SW_Push, SW57 SW_Push, SW58 SW_Push, SW59 SW_Push, SW6 SW_Push, SW60 SW_Push, SW61 SW_Push, SW62 SW_Push, SW63 SW_Push, SW64 SW_Push, SW7 SW_Push, SW8 SW_Push, SW9 SW_Push, U1 RaspberryPi_Pico, U2 RaspberryPi_Pico

Commit message: untested: learning from ai slop
Parts:
- U1: footprint Module:RaspberryPi_Pico_Common_THT -> ARGV:RaspberryPi_Pico_Case_THT
Changed lines of the file:
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@@
         (font
           (size 1.27 1.27))))
-    (property "Footprint" "Module:RaspberryPi_Pico_Common_THT"
+    (property "Footprint" "ARGV:RaspberryPi_Pico_Case_THT"
       (at 292.1 66.04 0)
       (effects
